Commit message: Update multiverse_parser

File: multiverse_ws/src/multiverse/multiverse_parser/examples/usd_to_urdf/urdf/box_scenario.urdf (robot description, URDF)
Before this commit: robot box_scenario, 5 links, 2 joints
Links:
- link box: geometry collision box size=0.005156 0.32 0.335; collision box size=0.005156 0.32 0.335
- link box_flap_1: geometry collision mesh filename=package://multiverse_parser/examples/usd_to_urdf/urdf/box_s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 scale=1.0000000000000002 1.0000000000000004 1.0000000000000002
- link box_flap_2: geometry collision mesh filename=package://multiverse_parser/examples/usd_to_urdf/urdf/box_s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 scale=1.0000000000000002 1.0000000000000004 1.0000000000000002
- link cat: geometry collision mesh filename=package://multiverse_parser/examples/usd_to_urdf/urdf/box_s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 scale=1.0 1.0 1.0
Joints:
- added joint box_joint: type fixed, parent world, child box, origin xyz=0.0 0.0 0.17 rpy=0.0 -0.0 0.0
- added joint cat_joint: type fixed, parent world, child cat, origin xyz=-0.09594 0.193951 0.5 rpy=0.0 -0.0 0.0
- joint box_flap_1_joint: origin xyz=0.17000000178813934 0.0 0.16599999368190765 rpy=0.0 -0.0 0.0 -> xyz=0.17000000178813934 0.0 0.16599999368190765 rpy=-1.5707963267948966 0.0 0.0
- joint box_flap_2_joint: origin xyz=-0.17000000178813934 0.0 0.1679999977350235 rpy=0.0 -0.0 0.0 -> xyz=-0.17000000178813934 0.0 0.1679999977350235 rpy=1.5707963267948966 -0.0 0.0

File: multiverse_ws/src/multiverse/multiverse_parser/examples/usd_to_urdf/urdf/kitchen.urdf (robot description, URDF)
Before this commit: robot kitchen, 26 links, 24 joints
Links:
- link fridge_area_lower_drawer_main: geometry collision mesh filename=package://multiverse_parser/examples/usd_to_urdf/urdf/kitch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 scale=1.0 1.0 0.9999999999999998; collision mesh filename=package://multiverse_parser/examples/usd_to_urdf/urdf/kitch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 scale=1.0 1.0 1.0
- link iai_fridge_door: geometry collision box size=0.01 0.35 0.065; collision box size=0.01 0.35 0.065
- link kitchen: geometry collision box size=0.29 0.5 0.01; collision box size=0.56 0.5 0.13
- link kitchen_island_left_lower_drawer_main: geometry collision mesh filename=package://multiverse_parser/examples/usd_to_urdf/urdf/kitch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 scale=1.0 1.0 0.9999999999999998; collision mesh filename=package://multiverse_parser/examples/usd_to_urdf/urdf/kitch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 scale=1.0 1.0 1.0
- link kitchen_island_left_upper_drawer_main: geometry collision mesh filename=package://multiverse_parser/examples/usd_to_urdf/urdf/kitch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 scale=1.0 1.0 0.9999999999999998; collision mesh filename=package://multiverse_parser/examples/usd_to_urdf/urdf/kitch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 scale=1.0 1.0 1.0
- link kitchen_island_middle_lower_drawer_main: geometry collision mesh filename=package://multiverse_parser/examples/usd_to_urdf/urdf/kitch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 scale=1.0 1.0 1.0; collision mesh filename=package://multiverse_parser/examples/usd_to_urdf/urdf/kitch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 scale=1.0 1.0000000000000002 1.0
- link kitchen_island_middle_upper_drawer_main: geometry collision mesh filename=package://multiverse_parser/examples/usd_to_urdf/urdf/kitch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 scale=1.0 1.0 1.0; collision mesh filename=package://multiverse_parser/examples/usd_to_urdf/urdf/kitch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 scale=1.0 1.0000000000000002 1.0
- link kitchen_island_right_lower_drawer_main: geometry collision mesh filename=package://multiverse_parser/examples/usd_to_urdf/urdf/kitch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 scale=1.0 1.0 0.9999999999999998; collision mesh filename=package://multiverse_parser/examples/usd_to_urdf/urdf/kitch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 scale=1.0 1.0 1.0
- link kitchen_island_right_upper_drawer_main: geometry collision mesh filename=package://multiverse_parser/examples/usd_to_urdf/urdf/kitch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 scale=1.0 1.0 0.9999999999999998; collision mesh filename=package://multiverse_parser/examples/usd_to_urdf/urdf/kitch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 scale=1.0 1.0 1.0
- link oven_area_area_left_drawer_main: geometry collision box size=0.025 0.3 1.33; collision box size=0.036 0.25 0.1
- link oven_area_area_middle_lower_drawer_main: geometry collision mesh filename=package://multiverse_parser/examples/usd_to_urdf/urdf/kitch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 scale=1.0 1.0 1.0; collision mesh filename=package://multiverse_parser/examples/usd_to_urdf/urdf/kitch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 scale=1.0 1.0 1.0
- link oven_area_area_middle_upper_drawer_main: geometry collision mesh filename=package://multiverse_parser/examples/usd_to_urdf/urdf/kitch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 scale=0.9999999999999999 0.9999999999999999 1.0; collision mesh filename=package://multiverse_parser/examples/usd_to_urdf/urdf/kitch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 scale=1.0 1.0000000000000002 1.0000000000000002
- link oven_area_area_right_drawer_main: geometry collision box size=0.025 0.3 1.33; collision box size=0.036 0.25 0.1
- link oven_area_oven_door: geometry collision mesh filename=package://multiverse_parser/examples/usd_to_urdf/urdf/kitch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 scale=0.9999999999999999 0.9999999999999999 0.9999999999999999; collision mesh filename=package://multiverse_parser/examples/usd_to_urdf/urdf/kitch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 scale=1.0 1.0 0.9999999999999999
- link oven_area_oven_knob_oven: geometry collision mesh filename=package://multiverse_parser/examples/usd_to_urdf/urdf/kitch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 scale=0.9999999999999999 0.9999999999999999 0.9999999999999999; collision mesh filename=package://multiverse_parser/examples/usd_to_urdf/urdf/kitch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 scale=0.9999999999999999 1.0 1.0
- link oven_area_oven_knob_stove_1: geometry collision mesh filename=package://multiverse_parser/examples/usd_to_urdf/urdf/kitch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 scale=0.9999999999999999 0.9999999999999999 0.9999999999999999; collision mesh filename=package://multiverse_parser/examples/usd_to_urdf/urdf/kitch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 scale=0.9999999999999999 1.0 1.0
- link oven_area_oven_knob_stove_2: geometry collision mesh filename=package://multiverse_parser/examples/usd_to_urdf/urdf/kitch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 scale=0.9999999999999999 0.9999999999999999 0.9999999999999999; collision mesh filename=package://multiverse_parser/examples/usd_to_urdf/urdf/kitch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 scale=0.9999999999999999 1.0 1.0
- link oven_area_oven_knob_stove_3: geometry collision mesh filename=package://multiverse_parser/examples/usd_to_urdf/urdf/kitch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 scale=0.9999999999999999 0.9999999999999999 0.9999999999999999; collision mesh filename=package://multiverse_parser/examples/usd_to_urdf/urdf/kitch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 scale=0.9999999999999999 1.0 1.0
- link oven_area_oven_knob_stove_4: geometry collision mesh filename=package://multiverse_parser/examples/usd_to_urdf/urdf/kitch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 scale=0.9999999999999999 0.9999999999999999 0.9999999999999999; collision mesh filename=package://multiverse_parser/examples/usd_to_urdf/urdf/kitch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 scale=0.9999999999999999 1.0 1.0
- link sink_area_dish_washer_door: geometry collision mesh filename=package://multiverse_parser/examples/usd_to_urdf/urdf/kitch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 scale=0.9999999999999999 0.9999999999999999 0.9999999999999999; collision mesh filename=package://multiverse_parser/examples/usd_to_urdf/urdf/kitch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 scale=1.0 1.0 1.0
- link sink_area_dish_washer_tray_bottom: geometry collision box size=0.005 0.5 0.17; collision box size=0.005 0.5 0.17
- link sink_area_left_bottom_drawer_main: geometry collision mesh filename=package://multiverse_parser/examples/usd_to_urdf/urdf/kitch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 scale=0.9999999999999999 0.9999999999999999 1.0; collision mesh filename=package://multiverse_parser/examples/usd_to_urdf/urdf/kitch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 scale=0.9999999999999999 1.0 1.0
- link sink_area_left_middle_drawer_main: geometry collision mesh filename=package://multiverse_parser/examples/usd_to_urdf/urdf/kitch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 scale=0.9999999999999999 0.9999999999999999 1.0; collision mesh filename=package://multiverse_parser/examples/usd_to_urdf/urdf/kitch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 scale=0.9999999999999999 1.0 1.0
- link sink_area_left_upper_drawer_main: geometry collision mesh filename=package://multiverse_parser/examples/usd_to_urdf/urdf/kitch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 scale=0.9999999999999999 0.9999999999999999 1.0; collision mesh filename=package://multiverse_parser/examples/usd_to_urdf/urdf/kitch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 scale=1.0 1.0 1.0
- link sink_area_trash_drawer_main: geometry collision mesh filename=package://multiverse_parser/examples/usd_to_urdf/urdf/kitch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 scale=1.0 1.0 1.0; collision mesh filename=package://multiverse_parser/examples/usd_to_urdf/urdf/kitch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 scale=1.0 1.0 1.0
Joints:
- added joint kitchen_joint: type fixed, parent world, child kitchen, origin xyz=0.0 0.0 0.0 rpy=0.0 -0.0 0.0
- joint fridge_area_lower_drawer_main_joint: limit lower=0.0 upper=0.008377580222319268 effort=1000 velocity=1000 -> lower=0.0 upper=0.47999998927116394 effort=1000 velocity=1000; origin xyz=1.5549999475479126 -1.0 0.32249999046325684 rpy=0.0 -0.0 3.141592653589793 -> xyz=1.5549999475479126 -1.0 0.32249999046325684 rpy=-3.141592653589793 1.5707963267948966 0.0
- joint iai_fridge_door_joint: limit lower=0.0 upper=0.0274156309615495 effort=1000 velocity=1000 -> lower=0.0 upper=1.5708000552204227 effort=1000 velocity=1000
- joint kitchen_island_left_lower_drawer_main_joint: limit lower=0.0 upper=0.008377580222319268 effort=1000 velocity=1000 -> lower=0.0 upper=0.47999998927116394 effort=1000 velocity=1000; origin xyz=-1.062999963760376 0.9491999745368958 0.24500000476837158 rpy=0.0 -0.0 0.0 -> xyz=-1.062999963760376 0.9491999745368958 0.24500000476837158 rpy=-0.0 1.5707963267948966 0.0
- joint kitchen_island_left_upper_drawer_main_joint: limit lower=0.0 upper=0.008377580222319268 effort=1000 velocity=1000 -> lower=0.0 upper=0.47999998927116394 effort=1000 velocity=1000; origin xyz=-1.062999963760376 0.9491999745368958 0.5350000262260437 rpy=0.0 -0.0 0.0 -> xyz=-1.062999963760376 0.9491999745368958 0.5350000262260437 rpy=-0.0 1.5707963267948966 0.0
- joint kitchen_island_middle_lower_drawer_main_joint: limit lower=0.0 upper=0.008377580222319268 effort=1000 velocity=1000 -> lower=0.0 upper=0.47999998927116394 effort=1000 velocity=1000; origin xyz=-1.062999963760376 1.7491999864578247 0.24500000476837158 rpy=0.0 -0.0 0.0 -> xyz=-1.062999963760376 1.7491999864578247 0.24500000476837158 rpy=-0.0 1.5707963267948966 0.0
- joint kitchen_island_middle_upper_drawer_main_joint: limit lower=0.0 upper=0.008377580222319268 effort=1000 velocity=1000 -> lower=0.0 upper=0.47999998927116394 effort=1000 velocity=1000; origin xyz=-1.062999963760376 1.7491999864578247 0.5350000262260437 rpy=0.0 -0.0 0.0 -> xyz=-1.062999963760376 1.7491999864578247 0.5350000262260437 rpy=-0.0 1.5707963267948966 0.0
- joint kitchen_island_right_lower_drawer_main_joint: limit lower=0.0 upper=0.008377580222319268 effort=1000 velocity=1000 -> lower=0.0 upper=0.47999998927116394 effort=1000 velocity=1000; origin xyz=-1.062999963760376 2.5492000579833984 0.24500000476837158 rpy=0.0 -0.0 0.0 -> xyz=-1.062999963760376 2.5492000579833984 0.24500000476837158 rpy=-0.0 1.5707963267948966 0.0
- joint kitchen_island_right_upper_drawer_main_joint: limit lower=0.0 upper=0.008377580222319268 effort=1000 velocity=1000 -> lower=0.0 upper=0.47999998927116394 effort=1000 velocity=1000; origin xyz=-1.062999963760376 2.5492000579833984 0.5350000262260437 rpy=0.0 -0.0 0.0 -> xyz=-1.062999963760376 2.5492000579833984 0.5350000262260437 rpy=-0.0 1.5707963267948966 0.0
- joint oven_area_area_left_drawer_main_joint: limit lower=0.0 upper=0.008377580222319268 effort=1000 velocity=1000 -> lower=0.0 upper=0.47999998927116394 effort=1000 velocity=1000; origin xyz=1.2649999856948853 2.380000114440918 0.824999988079071 rpy=0.0 -0.0 3.141592653589793 -> xyz=1.2649999856948853 2.380000114440918 0.824999988079071 rpy=-3.141592653589793 1.5707963267948966 0.0
- joint oven_area_area_middle_lower_drawer_main_joint: limit lower=0.0 upper=0.008377580222319268 effort=1000 velocity=1000 -> lower=0.0 upper=0.47999998927116394 effort=1000 velocity=1000; origin xyz=1.5549999475479126 1.9299999475479126 0.4399999976158142 rpy=0.0 -0.0 3.141592653589793 -> xyz=1.5549999475479126 1.9299999475479126 0.4399999976158142 rpy=-3.141592653589793 1.5707963267948966 0.0
- joint oven_area_area_middle_upper_drawer_main_joint: limit lower=0.0 upper=0.008377580222319268 effort=1000 velocity=1000 -> lower=0.0 upper=0.47999998927116394 effort=1000 velocity=1000; origin xyz=1.5549999475479126 1.9299999475479126 0.800000011920929 rpy=0.0 -0.0 3.141592653589793 -> xyz=1.5549999475479126 1.9299999475479126 0.800000011920929 rpy=-3.141592653589793 1.5707963267948966 0.0
- joint oven_area_area_right_drawer_main_joint: limit lower=0.0 upper=0.008377580222319268 effort=1000 velocity=1000 -> lower=0.0 upper=0.47999998927116394 effort=1000 velocity=1000; origin xyz=1.2649999856948853 1.4800000190734863 0.824999988079071 rpy=0.0 -0.0 3.141592653589793 -> xyz=1.2649999856948853 1.4800000190734863 0.824999988079071 rpy=-3.141592653589793 1.5707963267948966 0.0
- joint oven_area_oven_door_joint: limit lower=0.0 upper=0.0274156309615495 effort=1000 velocity=1000 -> lower=0.0 upper=1.5708000552204227 effort=1000 velocity=1000
- joint oven_area_oven_knob_oven_joint: limit lower=0.0 upper=0.05483109131434166 effort=1000 velocity=1000 -> lower=0.0 upper=3.1415899904287032 effort=1000 velocity=1000
- joint oven_area_oven_knob_stove_1_joint: limit lower=0.0 upper=0.05483109131434166 effort=1000 velocity=1000 -> lower=0.0 upper=3.1415899904287032 effort=1000 velocity=1000
- joint oven_area_oven_knob_stove_2_joint: limit lower=0.0 upper=0.05483109131434166 effort=1000 velocity=1000 -> lower=0.0 upper=3.1415899904287032 effort=1000 velocity=1000
- joint oven_area_oven_knob_stove_3_joint: limit lower=0.0 upper=0.05483109131434166 effort=1000 velocity=1000 -> lower=0.0 upper=3.1415899904287032 effort=1000 velocity=1000
- joint oven_area_oven_knob_stove_4_joint: limit lower=0.0 upper=0.05483109131434166 effort=1000 velocity=1000 -> lower=0.0 upper=3.1415899904287032 effort=1000 velocity=1000
- joint sink_area_dish_washer_door_joint: limit lower=0.0 upper=0.0274156309615495 effort=1000 velocity=1000 -> lower=0.0 upper=1.5708000552204227 effort=1000 velocity=1000
- joint sink_area_dish_washer_tray_main: limit lower=0.0 upper=0.008377580222319268 effort=1000 velocity=1000 -> lower=0.0 upper=0.47999998927116394 effort=1000 velocity=1000; origin xyz=1.6349999904632568 0.20000000298023224 0.6200000047683716 rpy=0.0 -0.0 3.141592653589793 -> xyz=1.6349999904632568 0.20000000298023224 0.6200000047683716 rpy=-3.141592653589793 1.5707963267948966 0.0
- joint sink_area_left_bottom_drawer_main_joint: limit lower=0.0 upper=0.008377580222319268 effort=1000 velocity=1000 -> lower=0.0 upper=0.47999998927116394 effort=1000 velocity=1000; origin xyz=1.5549999475479126 0.8999999761581421 0.23000000417232513 rpy=0.0 -0.0 3.141592653589793 -> xyz=1.5549999475479126 0.8999999761581421 0.23000000417232513 rpy=-3.141592653589793 1.5707963267948966 0.0
- joint sink_area_left_middle_drawer_main_joint: limit lower=0.0 upper=0.008377580222319268 effort=1000 velocity=1000 -> lower=0.0 upper=0.47999998927116394 effort=1000 velocity=1000; origin xyz=1.5549999475479126 0.8999999761581421 0.5299999713897705 rpy=0.0 -0.0 3.141592653589793 -> xyz=1.5549999475479126 0.8999999761581421 0.5299999713897705 rpy=-3.141592653589793 1.5707963267948966 0.0
- joint sink_area_left_upper_drawer_main_joint: limit lower=0.0 upper=0.008377580222319268 effort=1000 velocity=1000 -> lower=0.0 upper=0.47999998927116394 effort=1000 velocity=1000; origin xyz=1.5549999475479126 0.8999999761581421 0.7549999952316284 rpy=0.0 -0.0 3.141592653589793 -> xyz=1.5549999475479126 0.8999999761581421 0.7549999952316284 rpy=-3.141592653589793 1.5707963267948966 0.0
- joint sink_area_trash_drawer_main_joint: limit lower=0.0 upper=0.008377580222319268 effort=1000 velocity=1000 -> lower=0.0 upper=0.47999998927116394 effort=1000 velocity=1000; origin xyz=1.5549999475479126 -0.4000000059604645 0.39500001072883606 rpy=0.0 -0.0 3.141592653589793 -> xyz=1.5549999475479126 -0.4000000059604645 0.39500001072883606 rpy=-3.141592653589793 1.5707963267948966 0.0
