Commit message: Packing python scripts

File: multiverse_ws/src/multiverse_core/multiverse_parser/examples/usd_to_urdf/urdf/box_scenario.urdf (robot description, URDF)
Before this commit: robot box_scenario, 5 links, 4 joints
Joints:
- joint box_flap_1_joint: origin xyz=0.17000000178813934 0.0 0.16599999368190765 rpy=-1.5707963267948966 0.0 0.0 -> xyz=0.17 0.0 0.166 rpy=-1.5707961924360403 0.0 0.0
- joint box_flap_2_joint: origin xyz=-0.17000000178813934 0.0 0.1679999977350235 rpy=1.5707963267948966 -0.0 0.0 -> xyz=-0.17 0.0 0.168 rpy=1.5707961924360403 -0.0 0.0
