Commit message: Fix meshes for world

File: multiverse_ws/src/multiverse_core/multiverse_parser/examples/world_to_urdf/urdf/isr-testbed.urdf (robot description, URDF)
Before this commit: robot world, 64 links, 63 joints
Links:
- link wardrobe__wardrobe__base_link: geometry collision box size=1.0 0.72 2.0; visual mesh filename=package://multiverse_parser/examples/world_to_urdf/world/mo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 scale=1.0 1.0 1.0
Joints:
- joint wardrobe__wardrobe__base_link_joint: origin xyz=-2.65 2.44 0.0 rpy=1.57 0.0 1.57 -> xyz=-2.65 2.44 0.0 rpy=0.0 0.0 0.0
