Commit message: Fix kitchen

File: multiverse_ws/src/multiverse_core/multiverse_parser/examples/urdf_to_mjcf/urdf/kitchen.urdf (robot description, URDF)
Before this commit: robot kitchen, 26 links, 25 joints
Links:
- removed link kitchen
- added link kitchen_root, mass 0.0; collision box size=0.29 0.5 0.01; collision box size=0.56 0.5 0.13
Joints:
- joint fridge_area_lower_drawer_main_joint: parent kitchen -> kitchen_root
- joint iai_fridge_door_joint: parent kitchen -> kitchen_root
- joint kitchen_island_left_lower_drawer_main_joint: parent kitchen -> kitchen_root
- joint kitchen_island_left_upper_drawer_main_joint: parent kitchen -> kitchen_root
- joint kitchen_island_middle_lower_drawer_main_joint: parent kitchen -> kitchen_root
- joint kitchen_island_middle_upper_drawer_main_joint: parent kitchen -> kitchen_root
- joint kitchen_island_right_lower_drawer_main_joint: parent kitchen -> kitchen_root
- joint kitchen_island_right_upper_drawer_main_joint: parent kitchen -> kitchen_root
- joint kitchen_joint: child kitchen -> kitchen_root
- joint oven_area_area_left_drawer_main_joint: parent kitchen -> kitchen_root
- joint oven_area_area_middle_lower_drawer_main_joint: parent kitchen -> kitchen_root
- joint oven_area_area_middle_upper_drawer_main_joint: parent kitchen -> kitchen_root
- joint oven_area_area_right_drawer_main_joint: parent kitchen -> kitchen_root
- joint oven_area_oven_door_joint: parent kitchen -> kitchen_root
- joint oven_area_oven_knob_oven_joint: parent kitchen -> kitchen_root
- joint oven_area_oven_knob_stove_1_joint: parent kitchen -> kitchen_root
- joint oven_area_oven_knob_stove_2_joint: parent kitchen -> kitchen_root
- joint oven_area_oven_knob_stove_3_joint: parent kitchen -> kitchen_root
- joint oven_area_oven_knob_stove_4_joint: parent kitchen -> kitchen_root
- joint sink_area_dish_washer_door_joint: parent kitchen -> kitchen_root
- joint sink_area_dish_washer_tray_main: parent kitchen -> kitchen_root
- joint sink_area_left_bottom_drawer_main_joint: parent kitchen -> kitchen_root
- joint sink_area_left_middle_drawer_main_joint: parent kitchen -> kitchen_root
- joint sink_area_left_upper_drawer_main_joint: parent kitchen -> kitchen_root
- joint sink_area_trash_drawer_main_joint: parent kitchen -> kitchen_root
