Commit message: Add urdf_to_fbx

File: multiverse_ws/src/multiverse_core/multiverse_parser/examples/urdf_to_mjcf/urdf/box_scenario.urdf (robot description, URDF)
Before this commit: robot box_scenario, 5 links, 4 joints
Links:
- link box_flap_1: geometry collision mesh filename=package://multiverse_parser/examples/urdf_to_mjcf/urdf/box_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 scale=1.0000000000000002 1.0000000000000004 1.0000000000000002
- link box_flap_2: geometry collision mesh filename=package://multiverse_parser/examples/urdf_to_mjcf/urdf/box_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 scale=1.0000000000000002 1.0000000000000004 1.0000000000000002
- link cat: geometry collision mesh filename=package://multiverse_parser/examples/urdf_to_mjcf/urdf/box_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 scale=1.0 1.0 1.0

File: multiverse_ws/src/multiverse_core/multiverse_parser/examples/urdf_to_mjcf/urdf/kitchen.urdf (robot description, URDF)
Before this commit: robot kitchen, 26 links, 25 joints
Links:
- link fridge_area_lower_drawer_main: geometry collision mesh filename=package://multiverse_parser/examples/urdf_to_mjcf/urdf/kitc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 scale=1.0 1.0 0.9999999999999998; collision mesh filename=package://multiverse_parser/examples/urdf_to_mjcf/urdf/kitc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 scale=1.0 1.0 1.0
- link iai_fridge_door: geometry collision box size=0.01 0.35 0.065; collision box size=0.01 0.35 0.065
- link kitchen_island_left_lower_drawer_main: geometry collision mesh filename=package://multiverse_parser/examples/urdf_to_mjcf/urdf/kitc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 scale=1.0 1.0 0.9999999999999998; collision mesh filename=package://multiverse_parser/examples/urdf_to_mjcf/urdf/kitc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 scale=1.0 1.0 1.0
- link kitchen_island_left_upper_drawer_main: geometry collision mesh filename=package://multiverse_parser/examples/urdf_to_mjcf/urdf/kitc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 scale=1.0 1.0 0.9999999999999998; collision mesh filename=package://multiverse_parser/examples/urdf_to_mjcf/urdf/kitc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 scale=1.0 1.0 1.0
- link kitchen_island_middle_lower_drawer_main: geometry collision mesh filename=package://multiverse_parser/examples/urdf_to_mjcf/urdf/kitc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 scale=1.0 1.0 1.0; collision mesh filename=package://multiverse_parser/examples/urdf_to_mjcf/urdf/kitc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 scale=1.0 1.0000000000000002 1.0
- link kitchen_island_middle_upper_drawer_main: geometry collision mesh filename=package://multiverse_parser/examples/urdf_to_mjcf/urdf/kitc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 scale=1.0 1.0 1.0; collision mesh filename=package://multiverse_parser/examples/urdf_to_mjcf/urdf/kitc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 scale=1.0 1.0000000000000002 1.0
- link kitchen_island_right_lower_drawer_main: geometry collision mesh filename=package://multiverse_parser/examples/urdf_to_mjcf/urdf/kitc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 scale=1.0 1.0 0.9999999999999998; collision mesh filename=package://multiverse_parser/examples/urdf_to_mjcf/urdf/kitc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 scale=1.0 1.0 1.0
- link kitchen_island_right_upper_drawer_main: geometry collision mesh filename=package://multiverse_parser/examples/urdf_to_mjcf/urdf/kitc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 scale=1.0 1.0 0.9999999999999998; collision mesh filename=package://multiverse_parser/examples/urdf_to_mjcf/urdf/kitc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 scale=1.0 1.0 1.0
- link kitchen_root: geometry collision box size=0.29 0.5 0.01; collision box size=0.56 0.5 0.13
- link oven_area_area_left_drawer_main: geometry collision box size=0.025 0.3 1.33; collision box size=0.036 0.25 0.1
- link oven_area_area_middle_lower_drawer_main: geometry collision mesh filename=package://multiverse_parser/examples/urdf_to_mjcf/urdf/kitc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 scale=1.0 1.0 1.0; collision mesh filename=package://multiverse_parser/examples/urdf_to_mjcf/urdf/kitc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 scale=1.0 1.0 1.0
- link oven_area_area_middle_upper_drawer_main: geometry collision mesh filename=package://multiverse_parser/examples/urdf_to_mjcf/urdf/kitc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 scale=0.9999999999999999 0.9999999999999999 1.0; collision mesh filename=package://multiverse_parser/examples/urdf_to_mjcf/urdf/kitc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 scale=1.0 1.0000000000000002 1.0000000000000002
- link oven_area_area_right_drawer_main: geometry collision box size=0.025 0.3 1.33; collision box size=0.036 0.25 0.1
- link oven_area_oven_door: geometry collision mesh filename=package://multiverse_parser/examples/urdf_to_mjcf/urdf/kitc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 scale=0.9999999999999999 0.9999999999999999 0.9999999999999999; collision mesh filename=package://multiverse_parser/examples/urdf_to_mjcf/urdf/kitc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 scale=1.0 1.0 0.9999999999999999
- link oven_area_oven_knob_oven: geometry collision mesh filename=package://multiverse_parser/examples/urdf_to_mjcf/urdf/kitc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 scale=0.9999999999999999 0.9999999999999999 0.9999999999999999; collision mesh filename=package://multiverse_parser/examples/urdf_to_mjcf/urdf/kitc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 scale=0.9999999999999999 1.0 1.0
- link oven_area_oven_knob_stove_1: geometry collision mesh filename=package://multiverse_parser/examples/urdf_to_mjcf/urdf/kitc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 scale=0.9999999999999999 0.9999999999999999 0.9999999999999999; collision mesh filename=package://multiverse_parser/examples/urdf_to_mjcf/urdf/kitc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 scale=0.9999999999999999 1.0 1.0
- link oven_area_oven_knob_stove_2: geometry collision mesh filename=package://multiverse_parser/examples/urdf_to_mjcf/urdf/kitc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 scale=0.9999999999999999 0.9999999999999999 0.9999999999999999; collision mesh filename=package://multiverse_parser/examples/urdf_to_mjcf/urdf/kitc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 scale=0.9999999999999999 1.0 1.0
- link oven_area_oven_knob_stove_3: geometry collision mesh filename=package://multiverse_parser/examples/urdf_to_mjcf/urdf/kitc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 scale=0.9999999999999999 0.9999999999999999 0.9999999999999999; collision mesh filename=package://multiverse_parser/examples/urdf_to_mjcf/urdf/kitc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 scale=0.9999999999999999 1.0 1.0
- link oven_area_oven_knob_stove_4: geometry collision mesh filename=package://multiverse_parser/examples/urdf_to_mjcf/urdf/kitc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 scale=0.9999999999999999 0.9999999999999999 0.9999999999999999; collision mesh filename=package://multiverse_parser/examples/urdf_to_mjcf/urdf/kitc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 scale=0.9999999999999999 1.0 1.0
- link sink_area_dish_washer_door: geometry collision mesh filename=package://multiverse_parser/examples/urdf_to_mjcf/urdf/kitc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 scale=0.9999999999999999 0.9999999999999999 0.9999999999999999; collision mesh filename=package://multiverse_parser/examples/urdf_to_mjcf/urdf/kitc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 scale=1.0 1.0 1.0
- link sink_area_left_bottom_drawer_main: geometry collision mesh filename=package://multiverse_parser/examples/urdf_to_mjcf/urdf/kitc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 scale=0.9999999999999999 0.9999999999999999 1.0; collision mesh filename=package://multiverse_parser/examples/urdf_to_mjcf/urdf/kitc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 scale=0.9999999999999999 1.0 1.0
- link sink_area_left_middle_drawer_main: geometry collision mesh filename=package://multiverse_parser/examples/urdf_to_mjcf/urdf/kitc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 scale=0.9999999999999999 0.9999999999999999 1.0; collision mesh filename=package://multiverse_parser/examples/urdf_to_mjcf/urdf/kitc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 scale=0.9999999999999999 1.0 1.0
- link sink_area_left_upper_drawer_main: geometry collision mesh filename=package://multiverse_parser/examples/urdf_to_mjcf/urdf/kitc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 scale=0.9999999999999999 0.9999999999999999 1.0; collision mesh filename=package://multiverse_parser/examples/urdf_to_mjcf/urdf/kitc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 scale=1.0 1.0 1.0
- link sink_area_trash_drawer_main: geometry collision mesh filename=package://multiverse_parser/examples/urdf_to_mjcf/urdf/kitc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 scale=1.0 1.0 1.0; collision mesh filename=package://multiverse_parser/examples/urdf_to_mjcf/urdf/kitc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 scale=1.0 1.0 1.0
