Commit message: Clean up multiverse_parser

File: multiverse/tests/multiverse_parser/input/apartment/urdf/apartment.urdf (robot description, URDF)
Before this commit: robot apartment, 129 links, 128 joints
Links:
- removed link dishwasher_tray1
- removed link dishwasher_tray2
- removed link dishwasher_tray3
- link fridge_base: geometry collision box size=0.01564 0.469566 0.929316; collision box size=0.116796 0.469566 0.56255
- link sink_drawer1: geometry collision box size=0.016712 0.219652 0.34661; collision box size=0.016712 0.219652 0.34661
Joints:
- removed joint dishwasher_tray1_joint
- removed joint dishwasher_tray2_joint
- removed joint dishwasher_tray3_joint
