Commit message: Cleanup multiverse_parser

File: multiverse/modules/multiverse_parser/resources/input/tiago_dual/urdf/tiago_dual_1.urdf (robot description, URDF)
Before this commit: robot tiago_dual, 70 links, 69 joints
Links:
- link arm_left_5_link: geometry collision mesh filename=file://../meshes/stl/arm_5_collision_wrist_2017.stl scale=-1.0 -1.0 -1.0; visual mesh filename=file://../meshes/obj/arm_5-wrist-2017.obj scale=-1.0 -1.0 -1.0
- link arm_left_6_link: geometry collision mesh filename=file://../meshes/stl/arm_6_collision_wrist_2017.stl scale=-1.0 -1.0000000000000004 -1.0000000000000004; visual mesh filename=file://../meshes/obj/arm_6-wrist-2017.obj scale=-1.0 -1.0000000000000004 -1.0000000000000004
- link arm_right_5_link: geometry collision mesh filename=file://../meshes/stl/arm_5_collision_wrist_2017.stl scale=1.0 1.0 1.0; visual mesh filename=file://../meshes/obj/arm_5-wrist-2017.obj scale=1.0 1.0 1.0
- link arm_right_6_link: geometry collision mesh filename=file://../meshes/stl/arm_6_collision_wrist_2017.stl scale=1.0 1.0 1.0; visual mesh filename=file://../meshes/obj/arm_6-wrist-2017.obj scale=1.0 1.0 1.0

File: multiverse/modules/multiverse_parser/resources/input/tiago_dual/urdf/tiago_dual_2.urdf (robot description, URDF)
Before this commit: robot world, 70 links, 69 joints
Links:
- removed link arm_left_1_link
- removed link arm_left_2_link
- removed link arm_left_3_link
- removed link arm_left_4_link
- removed link arm_left_5_link
- removed link arm_left_6_link
- removed link arm_left_7_link
- removed link arm_left_tool_link
- removed link arm_right_1_link
- removed link arm_right_2_link
- removed link arm_right_3_link
- removed link arm_right_4_link
- removed link arm_right_5_link
- removed link arm_right_6_link
- removed link arm_right_7_link
- removed link arm_right_tool_link
- removed link base_antenna_left_link
- removed link base_antenna_right_link
- removed link base_cover_link
- removed link base_imu_link
- removed link base_laser_link
- removed link base_mic_back_left_link
- removed link base_mic_back_right_link
- removed link base_mic_front_left_link
- removed link base_mic_front_right_link
- removed link base_sonar_01_link
- removed link base_sonar_02_link
- removed link base_sonar_03_link
- removed link caster_back_left_1_link
- removed link caster_back_left_2_link
- removed link caster_back_right_1_link
- removed link caster_back_right_2_link
- removed link caster_front_left_1_link
- removed link caster_front_left_2_link
- removed link caster_front_right_1_link
- removed link caster_front_right_2_link
- removed link gripper_left_grasping_frame
- removed link gripper_left_left_finger_link
- removed link gripper_left_link
- removed link gripper_left_right_finger_link
- removed link gripper_left_tool_link
- removed link gripper_right_grasping_frame
- removed link gripper_right_left_finger_link
- removed link gripper_right_link
- removed link gripper_right_right_finger_link
- removed link gripper_right_tool_link
- removed link head_1_link
- removed link head_2_link
- removed link rgbd_laser_link
- removed link suspension_left_link
- removed link suspension_right_link
- removed link torso_fixed_column_link
- removed link torso_fixed_link
- removed link torso_lift_link
- removed link wheel_left_link
- removed link wheel_right_link
- removed link wrist_left_ft_link
- removed link wrist_left_ft_tool_link
- removed link wrist_right_ft_link
- removed link wrist_right_ft_tool_link
- removed link xtion_depth_frame
- removed link xtion_depth_optical_frame
- removed link xtion_link
- removed link xtion_optical_frame
- removed link xtion_orbbec_aux_joint_frame
- removed link xtion_rgb_frame
- removed link xtion_rgb_optical_frame
Joints:
- removed joint arm_left_1_joint
- removed joint arm_left_2_joint
- removed joint arm_left_3_joint
- removed joint arm_left_4_joint
- removed joint arm_left_5_joint
- removed joint arm_left_6_joint
- removed joint arm_left_7_joint
- removed joint arm_left_tool_link_joint
- removed joint arm_right_1_joint
- removed joint arm_right_2_joint
- removed joint arm_right_3_joint
- removed joint arm_right_4_joint
- removed joint arm_right_5_joint
- removed joint arm_right_6_joint
- removed joint arm_right_7_joint
- removed joint arm_right_tool_link_joint
- removed joint base_antenna_left_link_joint
- removed joint base_antenna_right_link_joint
- removed joint base_cover_link_joint
- removed joint base_imu_link_joint
- removed joint base_laser_link_joint
- removed joint base_mic_back_left_link_joint
- removed joint base_mic_back_right_link_joint
- removed joint base_mic_front_left_link_joint
- removed joint base_mic_front_right_link_joint
- removed joint base_sonar_01_link_joint
- removed joint base_sonar_02_link_joint
- removed joint base_sonar_03_link_joint
- removed joint caster_back_left_1_joint
- removed joint caster_back_left_2_joint
- removed joint caster_back_right_1_joint
- removed joint caster_back_right_2_joint
- removed joint caster_front_left_1_joint
- removed joint caster_front_left_2_joint
- removed joint caster_front_right_1_joint
- removed joint caster_front_right_2_joint
- removed joint gripper_left_grasping_frame_joint
- removed joint gripper_left_left_finger_joint
- removed joint gripper_left_link_joint
- removed joint gripper_left_right_finger_joint
- removed joint gripper_left_tool_link_joint
- removed joint gripper_right_grasping_frame_joint
- removed joint gripper_right_left_finger_joint
- removed joint gripper_right_link_joint
- removed joint gripper_right_right_finger_joint
- removed joint gripper_right_tool_link_joint
- removed joint head_1_joint
- removed joint head_2_joint
- removed joint rgbd_laser_link_joint
- removed joint suspension_left_joint
- removed joint suspension_right_joint
- removed joint torso_fixed_column_link_joint
- removed joint torso_fixed_link_joint
- removed joint torso_lift_joint
- removed joint wheel_left_joint
- removed joint wheel_right_joint
- removed joint wrist_left_ft_link_joint
- removed joint wrist_left_ft_tool_link_joint
- removed joint wrist_right_ft_link_joint
- removed joint wrist_right_ft_tool_link_joint
- removed joint xtion_depth_frame_joint
- removed joint xtion_depth_optical_frame_joint
- removed joint xtion_link_joint
- removed joint xtion_optical_frame_joint
- removed joint xtion_orbbec_aux_joint_frame_joint
- removed joint xtion_rgb_frame_joint
- removed joint xtion_rgb_optical_frame_joint
