Commit message: Update multiverse_parser

File: multiverse/modules/multiverse_parser/resources/input/tiago_dual/urdf/tiago_dual_2.urdf (robot description, URDF)
Before this commit: robot world, 3 links, 2 joints
Links:
- added link arm_left_1_link; collision mesh filename=file://../meshes/stl/arm_1_collision.stl scale=1.0 1.0000000000000004 1.0000000000000004; visual mesh filename=file://../meshes/obj/arm_1.obj scale=1.0 1.0000000000000004 1.0000000000000004
- added link torso_fixed_link; collision box size=0.25 0.25 0.1; collision box size=0.4 0.25 0.04
- added link torso_lift_link; collision mesh filename=file://../meshes/stl/torso_lift_collision_core.stl scale=1.0 1.0 1.0; collision mesh filename=file://../meshes/stl/torso_lift_collision_neck.stl scale=1.0 1.0 1.0
Joints:
- added joint arm_left_1_joint: type revolute, parent torso_lift_link, child arm_left_1_link, origin xyz=0.02556000091135502 0.1899999976158142 -0.17100000381469727 rpy=3.141592653589793 -0.0 1.5707963267948966, axis 0 0 1, limit lower=-1.1780972450961724 upper=1.5707963267948966 effort=1000 velocity=1000
- added joint torso_fixed_link_joint: type fixed, parent base_link, child torso_fixed_link, origin xyz=-0.062 0.0 0.193 rpy=0.0 -0.0 0.0
- added joint torso_lift_joint: type prismatic, parent torso_fixed_link, child torso_lift_link, origin xyz=0.0 0.0 0.597000002861023 rpy=0.0 -0.0 0.0, axis 0 0 1, limit lower=0.0 upper=0.800000011920929 effort=1000 velocity=1000
