Commit message: Update crane

File: multiverse/resources/robots/crane/urdf/crane.urdf (robot description, URDF)
Before this commit: robot crane_model, 39 links, 38 joints
Links:
- added link arm_cylinder_barrel_left, mass 23.5593; collision mesh filename=file://../meshes/collision/arm_cylinder_barrel_left_001.stl; collision mesh filename=file://../meshes/collision/arm_cylinder_barrel_left_002.stl
- added link arm_cylinder_barrel_right, mass 23.5593; collision mesh filename=file://../meshes/collision/arm_cylinder_barrel_right_001.stl; collision mesh filename=file://../meshes/collision/arm_cylinder_barrel_right_002.stl
- added link arm_cylinder_cover_left, mass 0.001; visual mesh filename=file://../meshes/visual/arm_cylinder_piston_cover_left.stl
- added link arm_cylinder_cover_right, mass 0.001; visual mesh filename=file://../meshes/visual/arm_cylinder_piston_cover_right.stl
- added link arm_cylinder_piston_left, mass 35.407; collision mesh filename=file://../meshes/collision/arm_cylinder_piston_left_001.stl; collision mesh filename=file://../meshes/collision/arm_cylinder_piston_left_002.stl
- added link arm_cylinder_piston_right, mass 35.407; collision mesh filename=file://../meshes/collision/arm_cylinder_piston_right_001.stl; collision mesh filename=file://../meshes/collision/arm_cylinder_piston_right_002.stl
- added link boom_cylinder_barrel, mass 56.105053; collision mesh filename=file://../meshes/collision/boom_cylinder_barrel.stl; visual mesh filename=file://../meshes/visual/boom_cylinder_barrel.stl
- added link boom_cylinder_cover, mass 0.001; visual mesh filename=file://../meshes/visual/boom_cylinder_piston_cover.stl
- added link boom_cylinder_linkage_big, mass 46.2496; collision mesh filename=file://../meshes/collision/boom_cylinder_linkage_big_001.stl; collision mesh filename=file://../meshes/collision/boom_cylinder_linkage_big_002.stl
- added link boom_cylinder_linkage_small, mass 11.392305; collision mesh filename=file://../meshes/collision/boom_cylinder_linkage_small_001.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; collision mesh filename=file://../meshes/collision/boom_cylinder_linkage_small_002.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
- added link boom_cylinder_piston, mass 52.359288; collision mesh filename=file://../meshes/collision/boom_cylinder_piston.stl; visual mesh filename=file://../meshes/visual/boom_cylinder_piston.stl
Joints:
- added joint arm_cylinder_mounting_on_boom_left: type revolute, parent K2_boom, child arm_cylinder_barrel_left, origin xyz=-1.6802 -0.0485 -0.224  rpy=0 0 -1.83314, axis 0 0 1, limit lower=-6 upper=6 effort=1000000000000 velocity=1000
- added joint arm_cylinder_mounting_on_boom_right: type revolute, parent K2_boom, child arm_cylinder_barrel_right, origin xyz=-1.6802 -0.0485 0.224  rpy=0 0 -1.83314, axis 0 0 1, limit lower=-6 upper=6 effort=1000000000000 velocity=1000
- added joint arm_cylinder_piston_in_barrel_linear_joint_left: type prismatic, parent arm_cylinder_barrel_left, child arm_cylinder_piston_left, origin xyz=0 1.617575 0 rpy=0 0 0, axis 0 1 0, limit lower=-0.373575 upper=0.5544250000000002 effort=3.3e5 velocity=1000
- added joint arm_cylinder_piston_in_barrel_linear_joint_right: type prismatic, parent arm_cylinder_barrel_right, child arm_cylinder_piston_right, origin xyz=0 1.617575 0 rpy=0 0 0, axis 0 1 0, limit lower=-0.373575 upper=0.5544250000000002 effort=3.3e5 velocity=1000
- added joint arm_piston_cover_left_mounting: type fixed, parent arm_cylinder_piston_left, child arm_cylinder_cover_left, origin xyz=0 0 0 rpy=0 0 0
- added joint arm_piston_cover_right_mounting: type fixed, parent arm_cylinder_piston_right, child arm_cylinder_cover_right, origin xyz=0 0 0 rpy=0 0 0
- added joint boom_cylinder_linkage_big_mounting_on_slewing_column: type revolute, parent K1_slewing_column, child boom_cylinder_linkage_big, origin xyz=-0.12 -0.07 0  rpy=0 0 -0.158245, axis 0 0 1, limit lower=-6 upper=6 effort=1000000000000 velocity=1000
- added joint boom_cylinder_linkage_small_mounting_on_boom: type revolute, parent K2_boom, child boom_cylinder_linkage_small, origin xyz=-3.039 -0.036034 0  rpy=0 0 -0.087064, axis 0 0 1, limit lower=-6 upper=6 effort=1000000000000 velocity=1000
- added joint boom_cylinder_mounting_on_slewing_column: type revolute, parent K1_slewing_column, child boom_cylinder_barrel, origin xyz=0.433 -1.7682 0  rpy=0 0 -0.00612, axis 0 0 1, limit lower=-6 upper=6 effort=1000000000000 velocity=1000
- added joint boom_cylinder_piston_in_barrel_linear_joint: type prismatic, parent boom_cylinder_barrel, child boom_cylinder_piston, origin xyz=0 0.43400700000000003 0  rpy=0 0 0, axis 0 1 0, limit lower=-0.36120700000000006 upper=0.6147930000000001 effort=4.4e5 velocity=1000
- added joint boom_piston_cover_mounting: type fixed, parent boom_cylinder_piston, child boom_cylinder_cover, origin xyz=0 0 0 rpy=0 0 0
