Commit message: Update multiverse_parser

File: multiverse/resources/worlds/isr_testbed/isr_testbed.urdf (robot description, URDF)
Before this commit: robot isr_testbed, 65 links, 64 joints
Links:
- removed link cone1__ConstructionCone__link
- removed link cone2__ConstructionCone__link
- removed link cone3__ConstructionCone__link
- removed link cone4__ConstructionCone__link
- removed link world
- added link cone1__Construction_Cone__link, mass 0.06330608576536179; collision mesh filename=file://isr_testbed/meshes/stl/construction_cone.stl scale=10.0 10.0 10.0
- added link cone2__Construction_Cone__link, mass 0.06330608576536179; collision mesh filename=file://isr_testbed/meshes/stl/construction_cone.stl scale=10.0 10.0 10.0
- added link cone3__Construction_Cone__link, mass 0.06330608576536179; collision mesh filename=file://isr_testbed/meshes/stl/construction_cone.stl scale=10.0 10.0 10.0
- added link cone4__Construction_Cone__link, mass 0.06330608576536179; collision mesh filename=file://isr_testbed/meshes/stl/construction_cone.stl scale=10.0 10.0 10.0
- link apple_juice_box__apple_juice__base_link: mass -4.690766886028541e-09 -> 1.2330989837646484; geometry collision box size=0.0689999982714653 0.0689999982714653 0.2590000033378601
- link aruco_marker_0__aruco_marker_0__link_0: mass 67.35200500488281 -> 67.35445404052734; geometry collision mesh filename=file://isr_testbed/meshes/stl/aruco_marker_0.stl scale=0.10000000149011612 0.10000000149011612 0.10000000149011612
- link basmati_rice__basmati_rice__base_link: mass -1.9402554229941416e-08 -> 0.8503400087356567; geometry collision box size=0.04100000113248825 0.12200000137090683 0.17000000178813934
- link bed__bed__link_0: mass 0.0034331518691033125 -> 2112.0; geometry collision box size=1.600000023841858 2.200000047683716 0.6000000238418579
- link beer__beer__link: geometry collision cylinder length=0.11999999731779099 radius=0.03500000014901161
- link cabinet_diamondback__cabinet_diamondback__base_link: mass -1.401834538228286e-06 -> 131.5006103515625; geometry collision mesh filename=file://isr_testbed/meshes/stl/cabinet_diamondback.stl scale=1.7999999523162842 1.0 1.0
- link cabinet_ikea_galant__cabinet_ikea_galant__base_link: mass -4.967053882865002e-06 -> 926.6400146484375; geometry collision box size=1.2999999523162842 0.5400000214576721 1.3200000524520874
- link chair1__tv_chair__link_0: mass -3.139732143608853e-05 -> 176.0; geometry collision box size=0.10000000149011612 0.10000000149011612 0.44999998807907104; collision box size=0.10000000149011612 0.10000000149011612 0.44999998807907104
- link chair2__tv_chair__link_0: mass -3.139732143608853e-05 -> 176.0; geometry collision box size=0.10000000149011612 0.10000000149011612 0.44999998807907104; collision box size=0.10000000149011612 0.10000000149011612 0.44999998807907104
- link chair_dinning_room_1__simple_chair__link_0: mass -2.1179857867537066e-06 -> 38.29999923706055; geometry collision box size=0.07999999821186066 0.07999999821186066 0.5; collision box size=0.07999999821186066 0.07999999821186066 0.5
- link chair_dinning_room_2__simple_chair__link_0: mass -2.1179857867537066e-06 -> 38.29999923706055; geometry collision box size=0.07999999821186066 0.07999999821186066 0.5; collision box size=0.07999999821186066 0.07999999821186066 0.5
- link chair_kitchen_1__simple_chair__link_0: mass -2.1179857867537066e-06 -> 38.29999923706055; geometry collision box size=0.07999999821186066 0.07999999821186066 0.5; collision box size=0.07999999821186066 0.07999999821186066 0.5
- link chair_kitchen_2__simple_chair__link_0: mass -2.1179857867537066e-06 -> 38.29999923706055; geometry collision box size=0.07999999821186066 0.07999999821186066 0.5; collision box size=0.07999999821186066 0.07999999821186066 0.5
- link chair_kitchen_3__simple_chair__link_0: mass -2.1179857867537066e-06 -> 38.29999923706055; geometry collision box size=0.07999999821186066 0.07999999821186066 0.5; collision box size=0.07999999821186066 0.07999999821186066 0.5
- link cup1__plastic_cup__link: mass 0.059198036789894104 -> 0.059198495000600815; geometry collision mesh filename=file://isr_testbed/meshes/stl/plastic_cup.stl scale=1.0 1.0 1.0
- link cup2__plastic_cup__link: mass 0.059198036789894104 -> 0.059198495000600815; geometry collision mesh filename=file://isr_testbed/meshes/stl/plastic_cup.stl scale=1.0 1.0 1.0
- link dinning_room_table__dinning_room_table__base_link: mass 0.00012353605416137725 -> 138.99114990234375; geometry collision box size=1.2999999523162842 0.8999999761581421 0.10000000149011612; collision cylinder length=0.699999988079071 radius=0.05000000074505806
- link human__person_standing__link: mass 144.47679138183594 -> 148.44007873535156; geometry collision box size=0.5 0.3499999940395355 0.019999999552965164; collision mesh filename=file://isr_testbed/meshes/stl/standing.stl scale=1.0 1.0 1.0
- link hydrant1__fire_hydrant__link: mass 36.59959411621094 -> 36.59939956665039; geometry collision mesh filename=file://isr_testbed/meshes/stl/fire_hydrant.stl scale=1.0 1.0 1.0
- link hydrant2__fire_hydrant__link: mass 36.59959411621094 -> 36.59939956665039; geometry collision mesh filename=file://isr_testbed/meshes/stl/fire_hydrant.stl scale=1.0 1.0 1.0
- link lamp_ikea_arstid__lamp_ikea_arstid__base_link: mass -1.0737880984379444e-07 -> 30.84415626525879; geometry collision cylinder length=0.019999999552965164 radius=0.18000000715255737; collision cylinder length=0.5 radius=0.12999999523162842
- link nightstand1__bedroom_nightstand__link_0: mass -1.140536642196821e-05 -> -149.60366821289062; geometry collision mesh filename=file://isr_testbed/meshes/stl/bedroom_nightstand.stl scale=1.0 1.0 1.0
- link nightstand2__bedroom_nightstand__link_0: mass -1.140536642196821e-05 -> -149.60366821289062; geometry collision mesh filename=file://isr_testbed/meshes/stl/bedroom_nightstand.stl scale=1.0 1.0 1.0
- link pizza_box__pizza_box__base_link: mass 1.5522043383953132e-07 -> 8.609999656677246; geometry collision box size=0.4099999964237213 0.6000000238418579 0.03500000014901161
- link plant_floor_small__plant_floor_small__base_link: mass -4.414080763126549e-07 -> 31.82853126525879; geometry collision mesh filename=file://isr_testbed/meshes/stl/plant_floor_small.stl scale=1.0 1.0 1.0
- link shelf__shelf__base_link: mass 936.5527954101562 -> 936.5327758789062; geometry collision mesh filename=file://isr_testbed/meshes/stl/shelf.stl scale=0.15000000596046448 0.20000000298023224 0.20000000298023224
- link sofa__sofa__link_0: mass 0.00015936137060634792 -> 1104.2030029296875; geometry collision box size=0.30000001192092896 1.8300000429153442 0.5; collision box size=0.800000011920929 0.25 0.5
- link table_bedside__table_bedside__base_link: mass 1.382431946694851e-07 -> 144.0; geometry collision box size=0.6000000238418579 0.6000000238418579 0.4000000059604645
- link table_living_room__table_living_room__base_link: mass 2.9766701118205674e-05 -> 221.1999969482422; geometry collision box size=0.11999999731779099 0.11999999731779099 0.75; collision box size=0.11999999731779099 0.11999999731779099 0.75
- link table_outside__cafe_table__link: mass -1.7171259969472885e-06 -> 41.983516693115234; geometry collision box size=0.041999999433755875 0.041999999433755875 0.150000005960464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; collision box size=0.5600000023841858 0.5600000023841858 0.03999999910593033
- link tea_box__tea_box__base_link: mass -9.701277114970708e-09 -> 0.7266420125961304; geometry collision box size=0.06300000101327896 0.15800000727176666 0.0729999989271164
- link tray_blue_white__tray_blue_white__base_link: mass -7.260799606001456e-08 -> 1.1039999723434448; geometry collision box size=0.23000000417232513 0.30000001192092896 0.01600000075995922
- link tree1__pine_tree__link: mass 91232.578125 -> 45616.28515625; geometry collision mesh filename=file://isr_testbed/meshes/stl/pine_tree.stl scale=1.0 1.0 1.0
- link tree2__pine_tree__link: mass 91232.578125 -> 45616.28515625; geometry collision mesh filename=file://isr_testbed/meshes/stl/pine_tree.stl scale=1.0 1.0 1.0
- link tv__tv__link_0: mass 3.275848257544567e-06 -> 288.0; geometry collision box size=0.30000001192092896 1.2000000476837158 0.800000011920929
- link tv_table__tv_table__link_0: mass -8.052059456531424e-06 -> 330.0; geometry collision box size=0.4000000059604645 1.649999976158142 0.5
- link wall__wall__Wall_0: geometry collision box size=16.5 0.15000000596046448 2.5
- link wall__wall__Wall_2: geometry collision box size=17.578399658203125 0.15000000596046448 2.5
- link walls__walls__Door_4: geometry collision box size=0.906000018119812 0.05000000074505806 1.2000000476837158
- link walls__walls__Wall_19: geometry collision box size=1.899999976158142 0.05000000074505806 1.0
- link walls__walls__Wall_21: geometry collision box size=2.1500000953674316 0.05000000074505806 1.2000000476837158
- link walls__walls__Wall_22: geometry collision box size=1.149999976158142 0.05000000074505806 1.2000000476837158
- link walls__walls__Wall_23: geometry collision box size=2.1500000953674316 0.05000000074505806 1.2000000476837158
- link walls__walls__Wall_24: geometry collision box size=1.149999976158142 0.05000000074505806 1.2000000476837158
- link walls__walls__Wall_25: geometry collision box size=0.6499999761581421 0.05000000074505806 1.2000000476837158
- link walls__walls__Wall_26: geometry collision box size=1.899999976158142 0.05000000074505806 1.2000000476837158
- link walls__walls__Wall_27: geometry collision box size=0.8999999761581421 0.05000000074505806 1.2000000476837158
- link walls__walls__Wall_36: geometry collision box size=1.899999976158142 0.05000000074505806 1.2000000476837158
- link walls__walls__Wall_48: geometry collision box size=8.900010108947754 0.05000000074505806 1.2000000476837158
- link walls__walls__Wall_49: geometry collision box size=4.650000095367432 0.05000000074505806 1.2000000476837158
- link walls__walls__Wall_50: geometry collision box size=2.4000000953674316 0.05000000074505806 1.2000000476837158
- link walls__walls__Wall_51: geometry collision box size=0.8999999761581421 0.05000000074505806 1.2000000476837158
- link walls__walls__Wall_53: geometry collision box size=3.4000000953674316 0.05000000074505806 1.2000000476837158
- link walls__walls__Wall_58: geometry collision box size=3.4000000953674316 0.05000000074505806 1.2000000476837158
- link walls__walls__Wall_61: geometry collision box size=2.6500000953674316 0.05000000074505806 1.2000000476837158
- link walls__walls__Wall_63: geometry collision box size=3.4000000953674316 0.05000000074505806 1.2000000476837158
- link wardrobe__wardrobe__base_link: mass 283.6346435546875 -> 1440.0; geometry collision box size=1.0 0.7200000286102295 2.0
Joints:
- removed joint cone1__ConstructionCone__link_joint
- removed joint cone2__ConstructionCone__link_joint
- removed joint cone3__ConstructionCone__link_joint
- removed joint cone4__ConstructionCone__link_joint
- removed joint world_joint
- added joint cone1__Construction_Cone__link_joint: type fixed, parent isr_testbed, child cone1__Construction_Cone__link, origin xyz=-5.94 2.97 0.0 rpy=0.0 0.0 0.0
- added joint cone2__Construction_Cone__link_joint: type fixed, parent isr_testbed, child cone2__Construction_Cone__link, origin xyz=-4.54 2.97 0.0 rpy=0.0 0.0 0.0
- added joint cone3__Construction_Cone__link_joint: type fixed, parent isr_testbed, child cone3__Construction_Cone__link, origin xyz=3.03 6.84 0.0 rpy=0.0 0.0 0.0
- added joint cone4__Construction_Cone__link_joint: type fixed, parent isr_testbed, child cone4__Construction_Cone__link, origin xyz=3.03 8.33 0.0 rpy=0.0 0.0 0.0
- joint apple_juice_box__apple_juice__base_link_joint: parent world -> isr_testbed
- joint aruco_marker_0__aruco_marker_0__link_0_joint: parent world -> isr_testbed
- joint basmati_rice__basmati_rice__base_link_joint: parent world -> isr_testbed
- joint bed__bed__link_0_joint: parent world -> isr_testbed
- joint beer__beer__link_joint: parent world -> isr_testbed
- joint cabinet_diamondback__cabinet_diamondback__base_link_joint: parent world -> isr_testbed
- joint cabinet_ikea_galant__cabinet_ikea_galant__base_link_joint: parent world -> isr_testbed
- joint chair1__tv_chair__link_0_joint: parent world -> isr_testbed
- joint chair2__tv_chair__link_0_joint: parent world -> isr_testbed
- joint chair_dinning_room_1__simple_chair__link_0_joint: parent world -> isr_testbed
- joint chair_dinning_room_2__simple_chair__link_0_joint: parent world -> isr_testbed
- joint chair_kitchen_1__simple_chair__link_0_joint: parent world -> isr_testbed
- joint chair_kitchen_2__simple_chair__link_0_joint: parent world -> isr_testbed
- joint chair_kitchen_3__simple_chair__link_0_joint: parent world -> isr_testbed
- joint cup1__plastic_cup__link_joint: parent world -> isr_testbed
- joint cup2__plastic_cup__link_joint: parent world -> isr_testbed
- joint dinning_room_table__dinning_room_table__base_link_joint: parent world -> isr_testbed
- joint human__person_standing__link_joint: parent world -> isr_testbed
- joint hydrant1__fire_hydrant__link_joint: parent world -> isr_testbed
- joint hydrant2__fire_hydrant__link_joint: parent world -> isr_testbed
- joint lamp_ikea_arstid__lamp_ikea_arstid__base_link_joint: parent world -> isr_testbed
- joint nightstand1__bedroom_nightstand__link_0_joint: parent world -> isr_testbed
- joint nightstand2__bedroom_nightstand__link_0_joint: parent world -> isr_testbed
- joint pizza_box__pizza_box__base_link_joint: parent world -> isr_testbed
- joint plant_floor_small__plant_floor_small__base_link_joint: parent world -> isr_testbed
- joint shelf__shelf__base_link_joint: parent world -> isr_testbed
- joint sofa__sofa__link_0_joint: parent world -> isr_testbed
- joint table_bedside__table_bedside__base_link_joint: parent world -> isr_testbed
- joint table_living_room__table_living_room__base_link_joint: parent world -> isr_testbed
- joint table_outside__cafe_table__link_joint: parent world -> isr_testbed
- joint tea_box__tea_box__base_link_joint: parent world -> isr_testbed
- joint tray_blue_white__tray_blue_white__base_link_joint: origin xyz=2.12 1.67 0.68 rpy=0.0 0.0 -1.5399999618530273 -> xyz=2.12 1.67 1.0 rpy=0.0 0.0 -1.5399999618530273; parent world -> isr_testbed
- joint tree1__pine_tree__link_joint: parent world -> isr_testbed
- joint tree2__pine_tree__link_joint: parent world -> isr_testbed
- joint tv__tv__link_0_joint: parent world -> isr_testbed
- joint tv_table__tv_table__link_0_joint: parent world -> isr_testbed
- joint wall_joint: parent world -> isr_testbed
- joint walls_joint: parent world -> isr_testbed
- joint wardrobe__wardrobe__base_link_joint: parent world -> isr_testbed
