Commit message: Add controller from mujoco

File: multiverse/resources/robots/universal_robot/ur5e/urdf/ur5e.urdf (robot description, URDF)
Before this commit: robot ur5e, 15 links, 14 joints
Links:
- removed link base
- removed link gripper_hand_e_base
- removed link gripper_hand_e_finger_1
- removed link gripper_hand_e_finger_2
Joints:
- removed joint base_joint
- removed joint gripper_hand_e_base_joint
- removed joint gripper_hand_e_finger_1_joint
- removed joint gripper_hand_e_finger_2_joint

Commit message: Update rviz2

File: multiverse/resources/robots/universal_robot/ur5e/urdf/ur5e.urdf (robot description, URDF)
Before this commit: robot ur5e, 11 links, 10 joints
Links:
- removed link base_link_inertia
- removed link flange
- removed link tool0
- removed link ur5e
- link base_link: mass None -> 4.0; geometry collision mesh filename=file://../meshes/stl/base.stl; visual mesh filename=file://../meshes/dae/base.dae
- link forearm_link: mass None -> 2.275; geometry collision mesh filename=file://../meshes/stl/forearm.stl; visual mesh filename=file://../meshes/dae/forearm.dae
- link shoulder_link: mass None -> 3.7; geometry collision mesh filename=file://../meshes/stl/shoulder.stl; visual mesh filename=file://../meshes/dae/shoulder.dae
- link upper_arm_link: mass None -> 8.393; geometry collision mesh filename=file://../meshes/stl/upperarm.stl; visual mesh filename=file://../meshes/dae/upperarm.dae
- link wrist_1_link: mass None -> 1.219; geometry collision mesh filename=file://../meshes/stl/wrist1.stl; visual mesh filename=file://../meshes/dae/wrist1.dae
- link wrist_2_link: mass None -> 1.219; geometry collision mesh filename=file://../meshes/stl/wrist2.stl; visual mesh filename=file://../meshes/dae/wrist2.dae
- link wrist_3_link: mass None -> 0.1879; geometry collision mesh filename=file://../meshes/stl/wrist3.stl; visual mesh filename=file://../meshes/dae/wrist3.dae
Joints:
- removed joint base_link_inertia_joint
- removed joint base_link_joint
- removed joint flange_joint
- removed joint tool0_joint
- joint elbow_joint: axis 0 0 1 -> 0 1 0; limit lower=0.0 upper=2.792526803190927 effort=1000 velocity=1000 -> lower=-3.141592653589793 upper=3.141592653589793 effort=150.0 velocity=3.14; origin xyz=-0.42500001192092896 0.0 0.0 rpy=0.0 -0.0 0.0 -> xyz=0.0 -0.131 0.425 rpy=0.0 0.0 0.0
- joint shoulder_lift_joint: axis 0 0 1 -> 0 1 0; limit lower=-3.141592653589793 upper=0.0 effort=1000 velocity=1000 -> lower=-6.283185307179586 upper=6.283185307179586 effort=150.0 velocity=3.14; origin xyz=0.0 0.0 0.0 rpy=1.5707963267948966 -0.0 0.0 -> xyz=0.0 0.138 0.0 rpy=0.0 1.5707963267948966 0.0
- joint shoulder_pan_joint: limit lower=0.0 upper=3.141592653589793 effort=1000 velocity=1000 -> lower=-6.283185307179586 upper=6.283185307179586 effort=150.0 velocity=3.14; origin xyz=0.0 0.0 0.16249999403953552 rpy=0.0 -0.0 0.0 -> xyz=0.0 0.0 0.163 rpy=0.0 0.0 0.0; parent base_link_inertia -> base_link
- joint wrist_1_joint: axis 0 0 1 -> 0 1 0; limit lower=-3.141592653589793 upper=1.3962634015954636 effort=1000 velocity=1000 -> lower=-6.283185307179586 upper=6.283185307179586 effort=28.0 velocity=6.28; origin xyz=-0.3921999931335449 0.0 0.13330000638961792 rpy=0.0 -0.0 0.0 -> xyz=0.0 0.0 0.392 rpy=0.0 1.5707963267948966 0.0
- joint wrist_2_joint: limit lower=-0.17453292519943295 upper=6.283185307179586 effort=1000 velocity=1000 -> lower=-6.283185307179586 upper=6.283185307179586 effort=28.0 velocity=6.28; origin xyz=0.0 -0.09969999641180038 -2.0448811047235615e-11 rpy=1.5707963267948966 -0.0 0.0 -> xyz=0.0 0.127 0.0 rpy=0.0 0.0 0.0
- joint wrist_3_joint: axis 0 0 1 -> 0 1 0; limit lower=-1.5707963267948966 upper=1.5707963267948966 effort=1000 velocity=1000 -> lower=-6.283185307179586 upper=6.283185307179586 effort=28.0 velocity=6.28; origin xyz=0.0 0.09960000216960907 -2.0428301411579142e-11 rpy=-1.5707963267948966 1.2246468260402848e-16 -1.2246468257891056e-16 -> xyz=0.0 0.0 0.1 rpy=0.0 0.0 0.0

Commit message: Fix some bugs

File: multiverse/resources/robots/universal_robot/ur5e/urdf/ur5e.urdf (robot description, URDF)
Before this commit: robot ur5e, 7 links, 6 joints
Links:
- link wrist_3_link: geometry collision mesh filename=file://../meshes/stl/wrist3.stl; visual mesh filename=file://../meshes/dae/wrist3.dae
