Commit message: Fix resources

File: multiverse/resources/robots/robotiq/gripper-2F-85/urdf/gripper-2F-85.urdf (robot description, URDF)
Before this commit: robot gripper-2F-85, 15 links, 14 joints
Links:
- link base: geometry collision mesh filename=file://../meshes/stl/base.stl scale=1.0 1.0 1.0; visual mesh filename=file://../meshes/obj/base.obj scale=1.0 1.0 1.0
- link base_mount: geometry collision mesh filename=file://../meshes/stl/base_mount.stl scale=1.0 1.0 1.0; visual mesh filename=file://../meshes/obj/base_mount.obj scale=1.0 1.0 1.0
- link gripper-2F-85: mass 0.0 -> None
- link left_coupler: geometry collision mesh filename=file://../meshes/stl/coupler.stl scale=1.0 1.0 1.0; visual mesh filename=file://../meshes/obj/coupler.obj scale=1.0 1.0 1.0
- link left_driver: geometry collision mesh filename=file://../meshes/stl/driver.stl scale=1.0 1.0 1.0; visual mesh filename=file://../meshes/obj/driver.obj scale=1.0 1.0 1.0
- link left_follower: geometry collision mesh filename=file://../meshes/stl/follower.stl scale=1.0 1.0 1.0; visual mesh filename=file://../meshes/obj/follower.obj scale=1.0 1.0 1.0
- link left_pad: geometry collision box size=0.02199999988079071 0.00800000037997961 0.01875000074505806; collision box size=0.02199999988079071 0.00800000037997961 0.01875000074505806
- link left_silicone_pad: geometry visual mesh filename=file://../meshes/obj/silicone_pad.obj scale=1.0 1.0 1.0
- link left_spring_link: geometry collision mesh filename=file://../meshes/stl/spring_link.stl scale=1.0 1.0 1.0; visual mesh filename=file://../meshes/obj/spring_link.obj scale=1.0 1.0 1.0
- link right_coupler: geometry collision mesh filename=file://../meshes/stl/coupler.stl scale=1.0 1.0 1.0; visual mesh filename=file://../meshes/obj/coupler.obj scale=1.0 1.0 1.0
- link right_driver: geometry collision mesh filename=file://../meshes/stl/driver.stl scale=1.0 1.0 1.0; visual mesh filename=file://../meshes/obj/driver.obj scale=1.0 1.0 1.0
- link right_follower: geometry collision mesh filename=file://../meshes/stl/follower.stl scale=1.0 1.0 1.0; visual mesh filename=file://../meshes/obj/follower.obj scale=1.0 1.0 1.0
- link right_pad: geometry collision box size=0.02199999988079071 0.00800000037997961 0.01875000074505806; collision box size=0.02199999988079071 0.00800000037997961 0.01875000074505806
- link right_silicone_pad: geometry visual mesh filename=file://../meshes/obj/silicone_pad.obj scale=1.0 1.0 1.0
- link right_spring_link: geometry collision mesh filename=file://../meshes/stl/spring_link.stl scale=1.0 1.0 1.0; visual mesh filename=file://../meshes/obj/spring_link.obj scale=1.0 1.0 1.0
Joints:
- joint base_joint: origin xyz=0.0 0.0 0.0038 rpy=0.0 0.0 -1.5707963267948966 -> xyz=0.0 0.0 0.0038 rpy=0.0 0.0 -1.5707963705062866
- joint base_mount_joint: origin xyz=0.0 0.0 0.007 rpy=0.0 -0.0 0.0 -> xyz=0.0 0.0 0.007 rpy=0.0 0.0 0.0
- joint left_coupler_joint: axis 1 0 0 -> 1.0 0.0 0.0; limit lower=-1.570000041628963 upper=0.0 effort=1000 velocity=1000 -> lower=-1.5700000524520874 upper=0.0 effort=1000.0 velocity=1000.0; origin xyz=0.0 0.03150000050663948 -0.004100000020116568 rpy=0.0 -0.0 0.0 -> xyz=0.0 0.03150000050663948 -0.004100000020116568 rpy=0.0 0.0 0.0
- joint left_driver_joint: axis 1 0 0 -> 1.0 0.0 0.0; limit lower=0.0 upper=255 effort=1000 velocity=1000 -> lower=0.0 upper=0.800000011920929 effort=1000.0 velocity=1000.0; origin xyz=0.0 -0.030601099133491516 0.05490399897098541 rpy=0.0 -0.0 3.141592653589793 -> xyz=0.0 -0.030601099133491516 0.05490399897098541 rpy=0.0 0.0 3.1415927410125732
- joint left_follower_joint: axis 1 0 0 -> 1.0 0.0 0.0; limit lower=-0.8726640267859195 upper=0.8726640267859195 effort=1000 velocity=1000 -> lower=-0.8726640343666077 upper=0.8726640343666077 effort=1000.0 velocity=1000.0; origin xyz=0.017999999225139618 0.054999999701976776 0.04399999976158142 rpy=0.0 -0.0 0.0 -> xyz=0.0 0.054999999701976776 0.03750000149011612 rpy=0.0 0.0 0.0
- joint left_pad_joint: origin xyz=0.0 -0.0189 0.01352 rpy=0.0 -0.0 0.0 -> xyz=0.0 -0.0189 0.01352 rpy=0.0 0.0 0.0
- joint left_silicone_pad_joint: origin xyz=0.0 0.0 0.0 rpy=0.0 -0.0 0.0 -> xyz=0.0 0.0 0.0 rpy=0.0 0.0 0.0
- joint left_spring_link_joint: axis 1 0 0 -> 1.0 0.0 0.0; limit lower=-0.29670597283903605 upper=0.8000000093382438 effort=1000 velocity=1000 -> lower=-0.296705961227417 upper=0.800000011920929 effort=1000.0 velocity=1000.0; origin xyz=3.851859888774472e-34 -0.013199999928474426 0.0608999989926815 rpy=0.0 -0.0 3.141592653589793 -> xyz=3.851859888774472e-34 -0.013199999928474426 0.0608999989926815 rpy=0.0 0.0 3.1415927410125732
- joint right_coupler_joint: axis 1 0 0 -> 1.0 0.0 0.0; limit lower=-1.570000041628963 upper=0.0 effort=1000 velocity=1000 -> lower=-1.5700000524520874 upper=0.0 effort=1000.0 velocity=1000.0; origin xyz=0.0 0.03150000050663948 -0.004100000020116568 rpy=0.0 -0.0 0.0 -> xyz=0.0 0.03150000050663948 -0.004100000020116568 rpy=0.0 0.0 0.0
- joint right_driver_joint: axis 1 0 0 -> 1.0 0.0 0.0; limit lower=0.0 upper=0.8000000093382438 effort=1000 velocity=1000 -> lower=0.0 upper=0.800000011920929 effort=1000.0 velocity=1000.0; mimic joint=left_driver_joint multiplier=1.0 offset=0.0 -> (none); origin xyz=0.0 0.030601099133491516 0.05490399897098541 rpy=0.0 -0.0 0.0 -> xyz=0.0 0.030601099133491516 0.05490399897098541 rpy=0.0 0.0 0.0
- joint right_follower_joint: axis 1 0 0 -> 1.0 0.0 0.0; limit lower=-0.8726640267859195 upper=0.8726640267859195 effort=1000 velocity=1000 -> lower=-0.8726640343666077 upper=0.8726640343666077 effort=1000.0 velocity=1000.0; origin xyz=-0.017999999225139618 0.054999999701976776 0.04399999976158142 rpy=0.0 -0.0 0.0 -> xyz=0.0 0.054999999701976776 0.03750000149011612 rpy=0.0 0.0 0.0
- joint right_pad_joint: origin xyz=0.0 -0.0189 0.01352 rpy=0.0 -0.0 0.0 -> xyz=0.0 -0.0189 0.01352 rpy=0.0 0.0 0.0
- joint right_silicone_pad_joint: origin xyz=0.0 0.0 0.0 rpy=0.0 -0.0 0.0 -> xyz=0.0 0.0 0.0 rpy=0.0 0.0 0.0
- joint right_spring_link_joint: axis 1 0 0 -> 1.0 0.0 0.0; limit lower=-0.29670597283903605 upper=0.8000000093382438 effort=1000 velocity=1000 -> lower=-0.296705961227417 upper=0.800000011920929 effort=1000.0 velocity=1000.0; origin xyz=-3.851859888774472e-34 0.013199999928474426 0.0608999989926815 rpy=0.0 -0.0 0.0 -> xyz=-3.851859888774472e-34 0.013199999928474426 0.0608999989926815 rpy=0.0 0.0 0.0

File: multiverse/resources/robots/universal_robot/ur5e/urdf/ur5e.urdf (robot description, URDF)
Before this commit: robot ur5e, 7 links, 6 joints
Links:
- link wrist_3_link: geometry collision mesh filename=file:///media/giangnguyen/Storage/Multiverse/multiverse/res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; visual mesh filename=file:///media/giangnguyen/Storage/Multiverse/multiverse/res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

Commit message: Fix gripper

File: multiverse/resources/robots/robotiq/gripper-2F-85/urdf/gripper-2F-85.urdf (robot description, URDF)
Before this commit: robot gripper-2F-85, 15 links, 14 joints
Links:
- removed link gripper-2F-85
- added link gripper_2F_85
- link base: geometry collision mesh filename=file://../meshes/stl/base.stl scale=1.0 1.0 1.0; visual mesh filename=file://../meshes/stl/base.stl scale=1.0 1.0 1.0
- link base_mount: geometry collision mesh filename=file://../meshes/stl/base_mount.stl scale=1.0 1.0 1.0; visual mesh filename=file://../meshes/stl/base_mount.stl scale=1.0 1.0 1.0
- link left_coupler: geometry collision mesh filename=file://../meshes/stl/coupler.stl scale=1.0 1.0 1.0; visual mesh filename=file://../meshes/stl/coupler.stl scale=1.0 1.0 1.0
- link left_driver: geometry collision mesh filename=file://../meshes/stl/driver.stl scale=1.0 1.0 1.0; visual mesh filename=file://../meshes/stl/driver.stl scale=1.0 1.0 1.0
- link left_follower: geometry collision mesh filename=file://../meshes/stl/follower.stl scale=1.0 1.0 1.0; visual mesh filename=file://../meshes/stl/follower.stl scale=1.0 1.0 1.0
- link left_silicone_pad: geometry visual mesh filename=file://../meshes/stl/silicone_pad.stl scale=1.0 1.0 1.0
- link left_spring_link: geometry collision mesh filename=file://../meshes/stl/spring_link.stl scale=1.0 1.0 1.0; visual mesh filename=file://../meshes/stl/spring_link.stl scale=1.0 1.0 1.0
- link right_coupler: geometry collision mesh filename=file://../meshes/stl/coupler.stl scale=1.0 1.0 1.0; visual mesh filename=file://../meshes/stl/coupler.stl scale=1.0 1.0 1.0
- link right_driver: geometry collision mesh filename=file://../meshes/stl/driver.stl scale=1.0 1.0 1.0; visual mesh filename=file://../meshes/stl/driver.stl scale=1.0 1.0 1.0
- link right_follower: geometry collision mesh filename=file://../meshes/stl/follower.stl scale=1.0 1.0 1.0; visual mesh filename=file://../meshes/stl/follower.stl scale=1.0 1.0 1.0
- link right_silicone_pad: geometry visual mesh filename=file://../meshes/stl/silicone_pad.stl scale=1.0 1.0 1.0
- link right_spring_link: geometry collision mesh filename=file://../meshes/stl/spring_link.stl scale=1.0 1.0 1.0; visual mesh filename=file://../meshes/stl/spring_link.stl scale=1.0 1.0 1.0
Joints:
- joint base_mount_joint: parent gripper-2F-85 -> gripper_2F_85
- joint left_follower_joint: origin xyz=0.0 0.054999999701976776 0.03750000149011612 rpy=0.0 0.0 0.0 -> xyz=0.0 0.03700000047683716 0.04399999976158142 rpy=0.0 0.0 0.0
- joint left_pad_joint: origin xyz=0.0 -0.0189 0.01352 rpy=0.0 0.0 0.0 -> xyz=0.0 -0.0009 0.00702 rpy=0.0 0.0 0.0
- joint right_follower_joint: origin xyz=0.0 0.054999999701976776 0.03750000149011612 rpy=0.0 0.0 0.0 -> xyz=0.0 0.03700000047683716 0.04399999976158142 rpy=0.0 0.0 0.0
- joint right_pad_joint: origin xyz=0.0 -0.0189 0.01352 rpy=0.0 0.0 0.0 -> xyz=0.0 -0.0009 0.00702 rpy=0.0 0.0 0.0

Commit message: Fix name

File: multiverse/resources/robots/robotiq/gripper-2F-85/urdf/gripper-2F-85.urdf (robot description, URDF)
Before this commit: robot gripper_2F_85, 15 links, 14 joints
Links:
- removed link gripper_2F_85
- added link gripper-2F-85
Joints:
- joint base_mount_joint: parent gripper_2F_85 -> gripper-2F-85
