Commit message: Restructure

File: multiverse/resources/robots/arm/urdf/arm.urdf (robot description, URDF)
Before this commit: robot arm, 7 links, 6 joints
Links:
- link BASE: geometry collision mesh filename=file://../assets/meshes/stl/BASE.stl; visual mesh filename=file://../assets/meshes/stl/BASE.stl
- link LINK1: geometry collision mesh filename=file://../assets/meshes/stl/LINK1.stl; visual mesh filename=file://../assets/meshes/stl/LINK1.stl
- link LINK2: geometry collision mesh filename=file://../assets/meshes/stl/LINK2.stl; visual mesh filename=file://../assets/meshes/stl/LINK2.stl
- link LINK3: geometry collision mesh filename=file://../assets/meshes/stl/LINK3.stl; visual mesh filename=file://../assets/meshes/stl/LINK3.stl
- link LINK4: geometry collision mesh filename=file://../assets/meshes/stl/LINK4.stl; visual mesh filename=file://../assets/meshes/stl/LINK4.stl
- link LINK5: geometry collision mesh filename=file://../assets/meshes/stl/LINK5.stl; visual mesh filename=file://../assets/meshes/stl/LINK5.stl

File: multiverse/resources/robots/franka_robotics/panda/urdf/panda.urdf (robot description, URDF)
Before this commit: robot panda, 12 links, 11 joints
Links:
- link hand: geometry collision mesh filename=file://assets/meshes/stl/hand_c.stl scale=1.0 1.0 1.0; visual mesh filename=file://assets/meshes/obj/hand_0.obj scale=1.0 1.0 1.0
- link left_finger: geometry collision box size=0.006000000052154064 0.004000000189989805 0.006000000052154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; collision box size=0.006000000052154064 0.004000000189989805 0.006000000052154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
- link link0: geometry collision mesh filename=file://assets/meshes/stl/link0_c.stl scale=1.0 1.0 1.0; visual mesh filename=file://assets/meshes/obj/link0_0.obj scale=1.0 1.0 1.0
- link link1: geometry collision mesh filename=file://assets/meshes/stl/link1_c.stl scale=1.0 1.0 1.0; visual mesh filename=file://assets/meshes/obj/link1.obj scale=1.0 1.0 1.0
- link link2: geometry collision mesh filename=file://assets/meshes/stl/link2_c.stl scale=1.0 1.0 1.0; visual mesh filename=file://assets/meshes/obj/link2.obj scale=1.0 1.0 1.0
- link link3: geometry collision mesh filename=file://assets/meshes/stl/link3_c.stl scale=1.0 1.0 1.0; visual mesh filename=file://assets/meshes/obj/link3_0.obj scale=1.0 1.0 1.0
- link link4: geometry collision mesh filename=file://assets/meshes/stl/link4_c.stl scale=1.0 1.0 1.0; visual mesh filename=file://assets/meshes/obj/link4_0.obj scale=1.0 1.0 1.0
- link link5: geometry collision mesh filename=file://assets/meshes/stl/link5_c0.stl scale=1.0 1.0 1.0; collision mesh filename=file://assets/meshes/stl/link5_c1.stl scale=1.0 1.0 1.0
- link link6: geometry collision mesh filename=file://assets/meshes/stl/link6_c.stl scale=1.0 1.0 1.0; visual mesh filename=file://assets/meshes/obj/link6_0.obj scale=1.0 1.0 1.0
- link link7: geometry collision mesh filename=file://assets/meshes/stl/link7_c.stl scale=1.0 1.0 1.0; visual mesh filename=file://assets/meshes/obj/link7_0.obj scale=1.0 1.0 1.0
- link right_finger: geometry collision box size=0.006000000052154064 0.004000000189989805 0.006000000052154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; collision box size=0.006000000052154064 0.004000000189989805 0.006000000052154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

File: multiverse/resources/robots/pal_robotics/tiago_dual/urdf/tiago_dual.urdf (robot description, URDF)
Before this commit: robot tiago_dual, 70 links, 69 joints
Links:
- link arm_left_1_link: geometry collision mesh filename=file://../assets/meshes/stl/arm_1_collision.stl scale=1.0 1.0 1.0; visual mesh filename=file://../assets/meshes/obj/arm_1.obj scale=1.0 1.0 1.0
- link arm_left_2_link: geometry collision mesh filename=file://../assets/meshes/stl/arm_2_collision.stl scale=-1.0 -1.0 -1.0; visual mesh filename=file://../assets/meshes/obj/arm_2.obj scale=-1.0 -1.0 -1.0
- link arm_left_3_link: geometry collision mesh filename=file://../assets/meshes/stl/arm_3_collision.stl scale=-1.0 -1.0 -1.0; visual mesh filename=file://../assets/meshes/obj/arm_3.obj scale=-1.0 -1.0 -1.0
- link arm_left_4_link: geometry collision mesh filename=file://../assets/meshes/stl/arm_4_collision.stl scale=-1.0 -1.0 -1.0; visual mesh filename=file://../assets/meshes/obj/arm_4.obj scale=-1.0 -1.0 -1.0
- link arm_left_5_link: geometry collision mesh filename=file://../assets/meshes/stl/arm_5_collision_wrist_2017.stl scale=-1.0 -1.0 -1.0; visual mesh filename=file://../assets/meshes/obj/arm_5_wrist_2017.obj scale=-1.0 -1.0 -1.0
- link arm_left_6_link: geometry collision mesh filename=file://../assets/meshes/stl/arm_6_collision_wrist_2017.stl scale=-1.0 -1.0 -1.0; visual mesh filename=file://../assets/meshes/obj/arm_6_wrist_2017.obj scale=-1.0 -1.0 -1.0
- link arm_right_1_link: geometry collision mesh filename=file://../assets/meshes/stl/arm_1_collision.stl scale=-1.0 -1.0 -1.0; visual mesh filename=file://../assets/meshes/obj/arm_1.obj scale=-1.0 -1.0 -1.0
- link arm_right_2_link: geometry collision mesh filename=file://../assets/meshes/stl/arm_2_collision.stl scale=1.0 1.0 1.0; visual mesh filename=file://../assets/meshes/obj/arm_2.obj scale=1.0 1.0 1.0
- link arm_right_3_link: geometry collision mesh filename=file://../assets/meshes/stl/arm_3_collision.stl scale=1.0 1.0 1.0; visual mesh filename=file://../assets/meshes/obj/arm_3.obj scale=1.0 1.0 1.0
- link arm_right_4_link: geometry collision mesh filename=file://../assets/meshes/stl/arm_4_collision.stl scale=1.0 1.0 1.0; visual mesh filename=file://../assets/meshes/obj/arm_4.obj scale=1.0 1.0 1.0
- link arm_right_5_link: geometry collision mesh filename=file://../assets/meshes/stl/arm_5_collision_wrist_2017.stl scale=1.0 1.0 1.0; visual mesh filename=file://../assets/meshes/obj/arm_5_wrist_2017.obj scale=1.0 1.0 1.0
- link arm_right_6_link: geometry collision mesh filename=file://../assets/meshes/stl/arm_6_collision_wrist_2017.stl scale=1.0 1.0 1.0; visual mesh filename=file://../assets/meshes/obj/arm_6_wrist_2017.obj scale=1.0 1.0 1.0
- link base_antenna_left_link: geometry collision cylinder length=0.17000000178813934 radius=0.004999999888241291; visual mesh filename=file://../assets/meshes/obj/antenna.obj scale=1.0 1.0 1.0
- link base_antenna_right_link: geometry collision cylinder length=0.17000000178813934 radius=0.004999999888241291; visual mesh filename=file://../assets/meshes/obj/antenna.obj scale=1.0 1.0 1.0
- link base_cover_link: geometry visual mesh filename=file://../assets/meshes/obj/base_ring.obj scale=1.0 1.0 1.0
- link base_laser_link: geometry visual mesh filename=file://../assets/meshes/obj/sick_tim551.obj scale=1.0 1.0 1.0
- link base_link: geometry collision mesh filename=file://../assets/meshes/stl/base_collision.stl scale=1.0 1.0 1.0; visual mesh filename=file://../assets/meshes/obj/base.obj scale=1.0 1.0 1.0
- link base_sonar_01_link: geometry visual mesh filename=file://../assets/meshes/obj/srf05.obj scale=1.0 1.0 1.0
- link base_sonar_02_link: geometry visual mesh filename=file://../assets/meshes/obj/srf05.obj scale=1.0 1.0 1.0
- link base_sonar_03_link: geometry visual mesh filename=file://../assets/meshes/obj/srf05.obj scale=1.0 1.0 1.0
- link caster_back_left_1_link: geometry visual mesh filename=file://../assets/meshes/obj/caster_1.obj scale=1.0 1.0 1.0
- link caster_back_left_2_link: geometry collision sphere radius=0.02500000037252903; visual mesh filename=file://../assets/meshes/obj/caster_2.obj scale=1.0 1.0 1.0
- link caster_back_right_1_link: geometry visual mesh filename=file://../assets/meshes/obj/caster_1.obj scale=1.0 1.0 1.0
- link caster_back_right_2_link: geometry collision sphere radius=0.02500000037252903; visual mesh filename=file://../assets/meshes/obj/caster_2.obj scale=1.0 1.0 1.0
- link caster_front_left_1_link: geometry visual mesh filename=file://../assets/meshes/obj/caster_1.obj scale=1.0 1.0 1.0
- link caster_front_left_2_link: geometry collision sphere radius=0.02500000037252903; visual mesh filename=file://../assets/meshes/obj/caster_2.obj scale=1.0 1.0 1.0
- link caster_front_right_1_link: geometry visual mesh filename=file://../assets/meshes/obj/caster_1.obj scale=1.0 1.0 1.0
- link caster_front_right_2_link: geometry collision sphere radius=0.02500000037252903; visual mesh filename=file://../assets/meshes/obj/caster_2.obj scale=1.0 1.0 1.0
- link gripper_left_left_finger_link: geometry collision box size=0.009999999776482582 0.05000000074505806 0.10999999940395355; visual mesh filename=file://../assets/meshes/obj/gripper_finger_link.obj scale=1.000092625617981 0.9999073147773743 1.0
- link gripper_left_link: geometry collision mesh filename=file://../assets/meshes/stl/gripper_link_collision.stl scale=1.0 1.0 1.0; visual mesh filename=file://../assets/meshes/obj/gripper_link.obj scale=1.0 1.0 1.0
- link gripper_left_right_finger_link: geometry collision box size=0.009999999776482582 0.05000000074505806 0.10999999940395355; visual mesh filename=file://../assets/meshes/obj/gripper_finger_link.obj scale=-1.000092625617981 -0.9999073147773743 1.0
- link gripper_right_left_finger_link: geometry collision box size=0.009999999776482582 0.05000000074505806 0.10999999940395355; visual mesh filename=file://../assets/meshes/obj/gripper_finger_link.obj scale=1.000092625617981 0.9999073147773743 1.0
- link gripper_right_link: geometry collision mesh filename=file://../assets/meshes/stl/gripper_link_collision.stl scale=1.0 1.0 1.0; visual mesh filename=file://../assets/meshes/obj/gripper_link.obj scale=1.0 1.0 1.0
- link gripper_right_right_finger_link: geometry collision box size=0.009999999776482582 0.05000000074505806 0.10999999940395355; visual mesh filename=file://../assets/meshes/obj/gripper_finger_link.obj scale=-1.000092625617981 -0.9999073147773743 1.0
- link head_1_link: geometry collision mesh filename=file://../assets/meshes/stl/head_1_collision.stl scale=1.0 1.0 1.0; visual mesh filename=file://../assets/meshes/obj/head_1.obj scale=1.0 1.0 1.0
- link head_2_link: geometry collision mesh filename=file://../assets/meshes/stl/head_2_collision.stl scale=1.0 1.0 1.0; visual mesh filename=file://../assets/meshes/obj/head_2.obj scale=1.0 1.0 1.0
- link torso_fixed_link: geometry collision box size=0.25 0.25 0.10000000149011612; collision box size=0.4000000059604645 0.25 0.03999999910593033
- link torso_lift_link: geometry collision mesh filename=file://../assets/meshes/stl/torso_lift_collision_core.stl scale=1.0 1.0 1.0; collision mesh filename=file://../assets/meshes/stl/torso_lift_collision_neck.stl scale=1.0 1.0 1.0
- link wheel_left_link: geometry collision sphere radius=0.09849999845027924; visual mesh filename=file://../assets/meshes/obj/wheel.obj scale=1.0 1.0 1.0
- link wheel_right_link: geometry collision sphere radius=0.09849999845027924; visual mesh filename=file://../assets/meshes/obj/wheel.obj scale=1.0 1.0 1.0

File: multiverse/resources/worlds/isr_testbed/urdf/isr_testbed.urdf (robot description, URDF)
Before this commit: robot isr_testbed, 64 links, 63 joints
Links:
- link aruco_marker_0__aruco_marker_0__link_0: geometry collision mesh filename=file://../assets/meshes/stl/aruco_marker_0.stl scale=0.10000000149011612 0.10000000149011612 0.10000000149011612
- link cabinet_diamondback__cabinet_diamondback__base_link: geometry collision mesh filename=file://../assets/meshes/stl/cabinet_diamondback.stl scale=1.7999999523162842 1.0 1.0
- link cone1__Construction_Cone__link: geometry collision mesh filename=file://../assets/meshes/stl/construction_cone.stl scale=10.0 10.0 10.0
- link cone2__Construction_Cone__link: geometry collision mesh filename=file://../assets/meshes/stl/construction_cone.stl scale=10.0 10.0 10.0
- link cone3__Construction_Cone__link: geometry collision mesh filename=file://../assets/meshes/stl/construction_cone.stl scale=10.0 10.0 10.0
- link cone4__Construction_Cone__link: geometry collision mesh filename=file://../assets/meshes/stl/construction_cone.stl scale=10.0 10.0 10.0
- link cup1__plastic_cup__link: geometry collision mesh filename=file://../assets/meshes/stl/plastic_cup.stl scale=1.0 1.0 1.0
- link cup2__plastic_cup__link: geometry collision mesh filename=file://../assets/meshes/stl/plastic_cup.stl scale=1.0 1.0 1.0
- link human__person_standing__link: geometry collision box size=0.5 0.3499999940395355 0.019999999552965164; collision mesh filename=file://../assets/meshes/stl/standing.stl scale=1.0 1.0 1.0
- link hydrant1__fire_hydrant__link: geometry collision mesh filename=file://../assets/meshes/stl/fire_hydrant.stl scale=1.0 1.0 1.0
- link hydrant2__fire_hydrant__link: geometry collision mesh filename=file://../assets/meshes/stl/fire_hydrant.stl scale=1.0 1.0 1.0
- link nightstand1__bedroom_nightstand__link_0: geometry collision mesh filename=file://../assets/meshes/stl/bedroom_nightstand.stl scale=1.0 1.0 1.0
- link nightstand2__bedroom_nightstand__link_0: geometry collision mesh filename=file://../assets/meshes/stl/bedroom_nightstand.stl scale=1.0 1.0 1.0
- link plant_floor_small__plant_floor_small__base_link: geometry collision mesh filename=file://../assets/meshes/stl/plant_floor_small.stl scale=1.0 1.0 1.0
- link shelf__shelf__base_link: geometry collision mesh filename=file://../assets/meshes/stl/shelf.stl scale=0.15000000596046448 0.20000000298023224 0.20000000298023224
- link tree1__pine_tree__link: geometry collision mesh filename=file://../assets/meshes/stl/pine_tree.stl scale=1.0 1.0 1.0
- link tree2__pine_tree__link: geometry collision mesh filename=file://../assets/meshes/stl/pine_tree.stl scale=1.0 1.0 1.0
