Commit message: Fix rollin-jutstin

File: multiverse/resources/robots/dlr/rollin_justin/urdf/rollin-justin.urdf (robot description, URDF)
Before this commit: robot justin, 64 links, 63 joints
Links:
- removed link justin__base_link
- removed link justin__head1
- removed link justin__head2
- removed link justin__left_1thumb1
- removed link justin__left_1thumb2
- removed link justin__left_1thumb3
- removed link justin__left_1thumb4
- removed link justin__left_1thumb_base
- removed link justin__left_2tip1
- removed link justin__left_2tip2
- removed link justin__left_2tip3
- removed link justin__left_2tip4
- removed link justin__left_2tip_base
- removed link justin__left_3middle1
- removed link justin__left_3middle2
- removed link justin__left_3middle3
- removed link justin__left_3middle4
- removed link justin__left_3middle_base
- removed link justin__left_4ring1
- removed link justin__left_4ring2
- removed link justin__left_4ring3
- removed link justin__left_4ring4
- removed link justin__left_4ring_base
- removed link justin__left_arm1
- removed link justin__left_arm2
- removed link justin__left_arm3
- removed link justin__left_arm4
- removed link justin__left_arm5
- removed link justin__left_arm6
- removed link justin__left_arm7
- removed link justin__left_palm
- removed link justin__right_1thumb1
- removed link justin__right_1thumb2
- removed link justin__right_1thumb3
- removed link justin__right_1thumb4
- removed link justin__right_1thumb_base
- removed link justin__right_2tip1
- removed link justin__right_2tip2
- removed link justin__right_2tip3
- removed link justin__right_2tip4
- removed link justin__right_2tip_base
- removed link justin__right_3middle1
- removed link justin__right_3middle2
- removed link justin__right_3middle3
- removed link justin__right_3middle4
- removed link justin__right_3middle_base
- removed link justin__right_4ring1
- removed link justin__right_4ring2
- removed link justin__right_4ring3
- removed link justin__right_4ring4
- removed link justin__right_4ring_base
- removed link justin__right_arm1
- removed link justin__right_arm2
- removed link justin__right_arm3
- removed link justin__right_arm4
- removed link justin__right_arm5
- removed link justin__right_arm6
- removed link justin__right_arm7
- removed link justin__right_palm
- removed link justin__torso1
- removed link justin__torso2
- removed link justin__torso3
- removed link justin__torso4
- removed link justin__world
- added link base_link, mass 145; collision mesh filename=file://geoms/dae/visual/base.dae scale=1 1 1; visual mesh filename=file://geoms/dae/visual/base.dae scale=1 1 1
- added link head1, mass 2; collision mesh filename=file://geoms/dae/visual/head1.dae scale=1 1 1; visual mesh filename=file://geoms/dae/visual/head1.dae scale=1 1 1
- added link head2, mass 3; collision mesh filename=file://geoms/dae/visual/head2.dae scale=1 1 1; visual mesh filename=file://geoms/dae/visual/head2.dae scale=1 1 1
- added link left_1thumb1
- added link left_1thumb2, mass 0.05; collision mesh filename=file://geoms/dae/visual/finger-phaprox.dae scale=1 1 1; visual mesh filename=file://geoms/dae/visual/finger-phaprox.dae scale=1 1 1
- added link left_1thumb3, mass 0.05; collision mesh filename=file://geoms/dae/visual/finger-phamed.dae scale=1 1 1; visual mesh filename=file://geoms/dae/visual/finger-phamed.dae scale=1 1 1
- added link left_1thumb4, mass 0.05; collision mesh filename=file://geoms/dae/visual/hii2_geh_phadist_gesamt_asm.dae scale=1 1 1; visual mesh filename=file://geoms/dae/visual/hii2_geh_phadist_gesamt_asm.dae scale=1 1 1
- added link left_1thumb_base, mass 0.05; visual mesh filename=file://geoms/dae/visual/finger-base.dae scale=1 1 1
- added link left_2tip1
- added link left_2tip2, mass 0.05; collision mesh filename=file://geoms/dae/visual/finger-phaprox.dae scale=1 1 1; visual mesh filename=file://geoms/dae/visual/finger-phaprox.dae scale=1 1 1
- added link left_2tip3, mass 0.05; collision mesh filename=file://geoms/dae/visual/finger-phamed.dae scale=1 1 1; visual mesh filename=file://geoms/dae/visual/finger-phamed.dae scale=1 1 1
- added link left_2tip4, mass 0.05; collision mesh filename=file://geoms/dae/visual/hii2_geh_phadist_gesamt_asm.dae scale=1 1 1; visual mesh filename=file://geoms/dae/visual/hii2_geh_phadist_gesamt_asm.dae scale=1 1 1
- added link left_2tip_base, mass 0.05; visual mesh filename=file://geoms/dae/visual/finger-base.dae scale=1 1 1
- added link left_3middle1
- added link left_3middle2, mass 0.05; collision mesh filename=file://geoms/dae/visual/finger-phaprox.dae scale=1 1 1; visual mesh filename=file://geoms/dae/visual/finger-phaprox.dae scale=1 1 1
- added link left_3middle3, mass 0.05; collision mesh filename=file://geoms/dae/visual/finger-phamed.dae scale=1 1 1; visual mesh filename=file://geoms/dae/visual/finger-phamed.dae scale=1 1 1
- added link left_3middle4, mass 0.05; collision mesh filename=file://geoms/dae/visual/hii2_geh_phadist_gesamt_asm.dae scale=1 1 1; visual mesh filename=file://geoms/dae/visual/hii2_geh_phadist_gesamt_asm.dae scale=1 1 1
- added link left_3middle_base, mass 0.05; collision mesh filename=file://geoms/dae/visual/finger-base.dae scale=1 1 1; visual mesh filename=file://geoms/dae/visual/finger-base.dae scale=1 1 1
- added link left_4ring1
- added link left_4ring2, mass 0.05; collision mesh filename=file://geoms/dae/visual/finger-phaprox.dae scale=1 1 1; visual mesh filename=file://geoms/dae/visual/finger-phaprox.dae scale=1 1 1
- added link left_4ring3, mass 0.05; collision mesh filename=file://geoms/dae/visual/finger-phamed.dae scale=1 1 1; visual mesh filename=file://geoms/dae/visual/finger-phamed.dae scale=1 1 1
- added link left_4ring4, mass 0.05; collision mesh filename=file://geoms/dae/visual/hii2_geh_phadist_gesamt_asm.dae scale=1 1 1; visual mesh filename=file://geoms/dae/visual/hii2_geh_phadist_gesamt_asm.dae scale=1 1 1
- added link left_4ring_base, mass 0.05; visual mesh filename=file://geoms/dae/visual/finger-base.dae scale=1 1 1
- added link left_arm1, mass 2.6371; collision mesh filename=file://geoms/dae/visual/left_arm1.dae scale=1 1 1; visual mesh filename=file://geoms/dae/visual/left_arm1.dae scale=1 1 1
- added link left_arm2, mass 2.3261934; collision mesh filename=file://geoms/dae/visual/left_arm2.dae scale=1 1 1; visual mesh filename=file://geoms/dae/visual/left_arm2.dae scale=1 1 1
- added link left_arm3, mass 2.293; collision mesh filename=file://geoms/dae/visual/left_arm3.dae scale=1 1 1; visual mesh filename=file://geoms/dae/visual/left_arm3.dae scale=1 1 1
- added link left_arm4, mass 2.2036950; collision mesh filename=file://geoms/dae/visual/left_arm4.dae scale=1 1 1; visual mesh filename=file://geoms/dae/visual/left_arm4.dae scale=1 1 1
- added link left_arm5, mass 0.7010105; collision mesh filename=file://geoms/dae/visual/left_arm5.dae scale=1 1 1; visual mesh filename=file://geoms/dae/visual/left_arm5.dae scale=1 1 1
- added link left_arm6, mass 1.6742; collision mesh filename=file://geoms/dae/visual/left_arm6.dae scale=1 1 1; visual mesh filename=file://geoms/dae/visual/left_arm6.dae scale=1 1 1
- added link left_arm7, mass 0.270; collision mesh filename=file://geoms/dae/visual/left_arm7.dae scale=1 1 1; visual mesh filename=file://geoms/dae/visual/left_arm7.dae scale=1 1 1
- added link left_palm, mass 1.40
- added link right_1thumb1
- added link right_1thumb2, mass 0.03; collision mesh filename=file://geoms/dae/visual/finger-phaprox.dae scale=1 1 1; visual mesh filename=file://geoms/dae/visual/finger-phaprox.dae scale=1 1 1
- added link right_1thumb3, mass 0.03; collision mesh filename=file://geoms/dae/visual/finger-phamed.dae scale=1 1 1; visual mesh filename=file://geoms/dae/visual/finger-phamed.dae scale=1 1 1
- added link right_1thumb4, mass 0.03; collision mesh filename=file://geoms/dae/visual/hii2_geh_phadist_gesamt_asm.dae scale=1 1 1; visual mesh filename=file://geoms/dae/visual/hii2_geh_phadist_gesamt_asm.dae scale=1 1 1
- added link right_1thumb_base, mass 0.05; visual mesh filename=file://geoms/dae/visual/finger-base.dae scale=1 1 1
- added link right_2tip1
- added link right_2tip2, mass 0.03; collision mesh filename=file://geoms/dae/visual/finger-phaprox.dae scale=1 1 1; visual mesh filename=file://geoms/dae/visual/finger-phaprox.dae scale=1 1 1
- added link right_2tip3, mass 0.03; collision mesh filename=file://geoms/dae/visual/finger-phamed.dae scale=1 1 1; visual mesh filename=file://geoms/dae/visual/finger-phamed.dae scale=1 1 1
- added link right_2tip4, mass 0.05; collision mesh filename=file://geoms/dae/visual/hii2_geh_phadist_gesamt_asm.dae scale=1 1 1; visual mesh filename=file://geoms/dae/visual/hii2_geh_phadist_gesamt_asm.dae scale=1 1 1
- added link right_2tip_base, mass 0.05; visual mesh filename=file://geoms/dae/visual/finger-base.dae scale=1 1 1
- added link right_3middle1
- added link right_3middle2, mass 0.03; collision mesh filename=file://geoms/dae/visual/finger-phaprox.dae scale=1 1 1; visual mesh filename=file://geoms/dae/visual/finger-phaprox.dae scale=1 1 1
- added link right_3middle3, mass 0.03; collision mesh filename=file://geoms/dae/visual/finger-phamed.dae scale=1 1 1; visual mesh filename=file://geoms/dae/visual/finger-phamed.dae scale=1 1 1
- added link right_3middle4, mass 0.03; collision mesh filename=file://geoms/dae/visual/hii2_geh_phadist_gesamt_asm.dae scale=1 1 1; visual mesh filename=file://geoms/dae/visual/hii2_geh_phadist_gesamt_asm.dae scale=1 1 1
- added link right_3middle_base, mass 0.05; visual mesh filename=file://geoms/dae/visual/finger-base.dae scale=1 1 1
- added link right_4ring1
- added link right_4ring2, mass 0.03; collision mesh filename=file://geoms/dae/visual/finger-phaprox.dae scale=1 1 1; visual mesh filename=file://geoms/dae/visual/finger-phaprox.dae scale=1 1 1
- added link right_4ring3, mass 0.03; collision mesh filename=file://geoms/dae/visual/finger-phamed.dae scale=1 1 1; visual mesh filename=file://geoms/dae/visual/finger-phamed.dae scale=1 1 1
- added link right_4ring4, mass 0.03; collision mesh filename=file://geoms/dae/visual/hii2_geh_phadist_gesamt_asm.dae scale=1 1 1; visual mesh filename=file://geoms/dae/visual/hii2_geh_phadist_gesamt_asm.dae scale=1 1 1
- added link right_4ring_base, mass 0.05; visual mesh filename=file://geoms/dae/visual/finger-base.dae scale=1 1 1
- added link right_arm1, mass 2.6371; collision mesh filename=file://geoms/dae/visual/right_arm1.dae scale=1 1 1; visual mesh filename=file://geoms/dae/visual/right_arm1.dae scale=1 1 1
- added link right_arm2, mass 2.3261934; collision mesh filename=file://geoms/dae/visual/right_arm2.dae scale=1 1 1; visual mesh filename=file://geoms/dae/visual/right_arm2.dae scale=1 1 1
- added link right_arm3, mass 2.293; collision mesh filename=file://geoms/dae/visual/right_arm3.dae scale=1 1 1; visual mesh filename=file://geoms/dae/visual/right_arm3.dae scale=1 1 1
- added link right_arm4, mass 2.203695; collision mesh filename=file://geoms/dae/visual/right_arm4.dae scale=1 1 1; visual mesh filename=file://geoms/dae/visual/right_arm4.dae scale=1 1 1
- added link right_arm5, mass 0.7010105; collision mesh filename=file://geoms/dae/visual/right_arm5.dae scale=1 1 1; visual mesh filename=file://geoms/dae/visual/right_arm5.dae scale=1 1 1
- added link right_arm6, mass 1.6742; collision mesh filename=file://geoms/dae/visual/right_arm6.dae scale=1 1 1; visual mesh filename=file://geoms/dae/visual/right_arm6.dae scale=1 1 1
- added link right_arm7, mass 0.270; collision mesh filename=file://geoms/dae/visual/right_arm7.dae scale=1 1 1; visual mesh filename=file://geoms/dae/visual/right_arm7.dae scale=1 1 1
- added link right_palm, mass 1.40
- added link torso1, mass 4.554854; collision mesh filename=file://geoms/dae/visual/torso1.dae scale=1 1 1; visual mesh filename=file://geoms/dae/visual/torso1.dae scale=1 1 1
- added link torso2, mass 5.4703718; collision mesh filename=file://geoms/dae/visual/torso2.dae scale=1 1 1; visual mesh filename=file://geoms/dae/visual/torso2.dae scale=1 1 1
- added link torso3, mass 2.9250956; collision mesh filename=file://geoms/dae/visual/torso3.dae scale=1 1 1; visual mesh filename=file://geoms/dae/visual/torso3.dae scale=1 1 1
- added link torso4, mass 5.7594877; collision mesh filename=file://geoms/dae/visual/torso4.dae scale=1 1 1; visual mesh filename=file://geoms/dae/visual/torso4.dae scale=1 1 1
Joints:
- removed joint justin__fixed_to_ground
- removed joint justin__head1
- removed joint justin__head2
- removed joint justin__left_1thumb1
- removed joint justin__left_1thumb2
- removed joint justin__left_1thumb3
- removed joint justin__left_1thumb4
- removed joint justin__left_1thumb_base
- removed joint justin__left_2tip1
- removed joint justin__left_2tip2
- removed joint justin__left_2tip3
- removed joint justin__left_2tip4
- removed joint justin__left_2tip_base
- removed joint justin__left_3middle1
- removed joint justin__left_3middle2
- removed joint justin__left_3middle3
- removed joint justin__left_3middle4
- removed joint justin__left_3middle_base
- removed joint justin__left_4ring1
- removed joint justin__left_4ring2
- removed joint justin__left_4ring3
- removed joint justin__left_4ring4
- removed joint justin__left_4ring_base
- removed joint justin__left_arm1
- removed joint justin__left_arm2
- removed joint justin__left_arm3
- removed joint justin__left_arm4
- removed joint justin__left_arm5
- removed joint justin__left_arm6
- removed joint justin__left_arm7
- removed joint justin__left_palm
- removed joint justin__right_1thumb1
- removed joint justin__right_1thumb2
- removed joint justin__right_1thumb3
- removed joint justin__right_1thumb4
- removed joint justin__right_1thumb_base
- removed joint justin__right_2tip1
- removed joint justin__right_2tip2
- removed joint justin__right_2tip3
- removed joint justin__right_2tip4
- removed joint justin__right_2tip_base
- removed joint justin__right_3middle1
- removed joint justin__right_3middle2
- removed joint justin__right_3middle3
- removed joint justin__right_3middle4
- removed joint justin__right_3middle_base
- removed joint justin__right_4ring1
- removed joint justin__right_4ring2
- removed joint justin__right_4ring3
- removed joint justin__right_4ring4
- removed joint justin__right_4ring_base
- removed joint justin__right_arm1
- removed joint justin__right_arm2
- removed joint justin__right_arm3
- removed joint justin__right_arm4
- removed joint justin__right_arm5
- removed joint justin__right_arm6
- removed joint justin__right_arm7
- removed joint justin__right_palm
- removed joint justin__torso1
- removed joint justin__torso2
- removed joint justin__torso3
- removed joint justin__torso4
- added joint head1: type revolute, parent torso4, child head1, origin xyz=0.235  0.088  0 rpy=1.57079  0       1.57079, axis 0  0  1, limit lower=-0.785398 upper=0.785398 effort=150.0 velocity=0.85
- added joint head2: type revolute, parent head1, child head2, origin xyz=0  0  0 rpy=-1.57079  0       0, axis 0  0  1, limit lower=-0.436332 upper=0.785398 effort=150.0 velocity=0.85
- added joint left_1thumb1: type revolute, parent left_1thumb_base, child left_1thumb1, axis 0 0 1, limit lower=-0.523599 upper=0.523599 effort=3.5 velocity=0.85
- added joint left_1thumb2: type revolute, parent left_1thumb1, child left_1thumb2, origin xyz=0  0  0 rpy=1.57079  0       0, axis 0 0 1, limit lower=-0.349066 upper=1.50098 effort=3.5 velocity=0.85
- added joint left_1thumb3: type revolute, parent left_1thumb2, child left_1thumb3, origin xyz=0.075  0     0 rpy=0  0  0, axis 0 0 1, limit lower=-0.174533 upper=1.76278 effort=1.75 velocity=0.85
- added joint left_1thumb4: type revolute, parent left_1thumb3, child left_1thumb4, origin xyz=0.03999  0       0 rpy=0       0      -1.57079, axis 0 0 1, limit lower=-0.174533 upper=1.76278 effort=1.75 velocity=0.85, mimic joint=left_1thumb3 multiplier=1 offset=0
- added joint left_1thumb_base: type fixed, parent left_arm7, child left_1thumb_base, origin xyz=-0.0504  0.2029 -0.0462 rpy=1.34429  0.02834  2.14927, axis 0 0 1
- added joint left_2tip1: type revolute, parent left_2tip_base, child left_2tip1, axis 0 0 1, limit lower=-0.523599 upper=0.523599 effort=3.5 velocity=0.85
- added joint left_2tip2: type revolute, parent left_2tip1, child left_2tip2, origin xyz=0  0  0 rpy=1.57079  0       0, axis 0 0 1, limit lower=-0.349066 upper=1.50098 effort=3.5 velocity=0.85
- added joint left_2tip3: type revolute, parent left_2tip2, child left_2tip3, origin xyz=0.075  0     0 rpy=0  0  0, axis 0 0 1, limit lower=-0.174533 upper=1.76278 effort=1.75 velocity=0.85
- added joint left_2tip4: type revolute, parent left_2tip3, child left_2tip4, origin xyz=0.04  0    0 rpy=0       0      -1.57079, axis 0 0 1, limit lower=-0.174533 upper=1.76278 effort=1.75 velocity=0.85, mimic joint=left_2tip3 multiplier=1.0 offset=0
- added joint left_2tip_base: type fixed, parent left_arm7, child left_2tip_base, origin xyz=0.0482  0.2409 -0.0236 rpy=-1.69632 -0.11527  1.36803, axis 0 0 1
- added joint left_3middle1: type revolute, parent left_3middle_base, child left_3middle1, axis 0 0 1, limit lower=-0.523599 upper=0.523599 effort=3.5 velocity=0.85
- added joint left_3middle2: type revolute, parent left_3middle1, child left_3middle2, origin xyz=0  0  0 rpy=1.57079  0       0, axis 0 0 1, limit lower=-0.349066 upper=1.50098 effort=3.5 velocity=0.85
- added joint left_3middle3: type revolute, parent left_3middle2, child left_3middle3, origin xyz=0.07499  0       0 rpy=0  0  0, axis 0 0 1, limit lower=-0.174533 upper=1.76278 effort=1.75 velocity=0.85
- added joint left_3middle4: type revolute, parent left_3middle3, child left_3middle4, origin xyz=0.04  0    0 rpy=0       0      -1.57079, axis 0 0 1, limit lower=-0.174533 upper=1.76278 effort=1.75 velocity=0.85, mimic joint=left_3middle3 multiplier=1 offset=0
- added joint left_3middle_base: type fixed, parent left_arm7, child left_3middle_base, origin xyz=0.0469   0.2353   0.01629 rpy=-1.69632 -0.11527  1.36803, axis 0 0 1
- added joint left_4ring1: type revolute, parent left_4ring_base, child left_4ring1, axis 0 0 1, limit lower=-0.523599 upper=0.523599 effort=3.5 velocity=0.85
- added joint left_4ring2: type revolute, parent left_4ring1, child left_4ring2, origin xyz=0  0  0 rpy=1.57079  0       0, axis 0 0 1, limit lower=-0.349066 upper=1.50098 effort=3.5 velocity=0.85
- added joint left_4ring3: type revolute, parent left_4ring2, child left_4ring3, origin xyz=0.075  0     0 rpy=0  0  0, axis 0 0 1, limit lower=-0.174533 upper=1.76278 effort=1.75 velocity=0.85
- added joint left_4ring4: type revolute, parent left_4ring3, child left_4ring4, origin xyz=0.04  0    0 rpy=0       0      -1.57079, axis 0 0 1, limit lower=-0.174533 upper=1.76278 effort=1.75 velocity=0.85, mimic joint=left_4ring3 multiplier=1 offset=0
- added joint left_4ring_base: type fixed, parent left_arm7, child left_4ring_base, origin xyz=0.0374  0.2299  0.0623 rpy=-1.69632 -0.11527  1.36803, axis 0 0 1
- added joint left_arm1: type revolute, parent torso4, child left_arm1, origin xyz=0.19   0.088  0.256 rpy=-3.14159  0.52359  0, axis 0  0  1, limit lower=-2.96706 upper=2.96706 effort=150.0 velocity=0.85
- added joint left_arm2: type revolute, parent left_arm1, child left_arm2, origin xyz=0  0  0 rpy=1.57079  0       0, axis 0  0  1, limit lower=-2.0944 upper=2.0944 effort=150.0 velocity=0.85
- added joint left_arm3: type revolute, parent left_arm2, child left_arm3, origin xyz=0  -0.4  0 rpy=-2.87979 -1.57079  1.30899, axis 0  0 1, limit lower=-2.96706 upper=2.96706 effort=150.0 velocity=0.85
- added joint left_arm4: type revolute, parent left_arm3, child left_arm4, origin xyz=0  0  0 rpy=1.57079  0       0, axis 0 0 1, limit lower=-2.0944 upper=2.0944 effort=150.0 velocity=0.85
- added joint left_arm5: type revolute, parent left_arm4, child left_arm5, origin xyz=0   -0.39  0 rpy=-1.57079  0       0, axis 0 0 1, limit lower=-2.96706 upper=2.96706 effort=150.0 velocity=0.85
- added joint left_arm6: type revolute, parent left_arm5, child left_arm6, origin xyz=0  0  0 rpy=-0.71372  1.57079  0.85707, axis 0 0 1, limit lower=-0.785398 upper=1.39626 effort=150.0 velocity=0.85
- added joint left_arm7: type revolute, parent left_arm6, child left_arm7, origin xyz=0  0  0 rpy=-1.11887 -1.57079 -0.45192, axis 0 0 1, limit lower=-0.785398 upper=2.35619 effort=150.0 velocity=0.85
- added joint left_palm: type fixed, parent left_arm7, child left_palm, origin xyz=0  0.1011  0 rpy=1.57079 0.0 3.14159
- added joint right_1thumb1: type revolute, parent right_1thumb_base, child right_1thumb1, axis 0 0 1, limit lower=-0.523599 upper=0.523599 effort=3.5 velocity=0.85
- added joint right_1thumb2: type revolute, parent right_1thumb1, child right_1thumb2, origin xyz=0  0  0 rpy=1.57079  0       0, axis 0 0 1, limit lower=-0.349066 upper=1.50098 effort=3.5 velocity=0.85
- added joint right_1thumb3: type revolute, parent right_1thumb2, child right_1thumb3, origin xyz=0.075  0     0 rpy=0  0  0, axis 0 0 1, limit lower=-0.174533 upper=1.76278 effort=1.75 velocity=0.85
- added joint right_1thumb4: type revolute, parent right_1thumb3, child right_1thumb4, origin xyz=0.04  0    0 rpy=0       0      -1.57079, axis 0 0 1, limit lower=-0.174533 upper=1.76278 effort=1.75 velocity=0.85, mimic joint=right_1thumb3 multiplier=1.0 offset=0
- added joint right_1thumb_base: type fixed, parent right_arm7, child right_1thumb_base, origin xyz=-0.0504  0.2029  0.0462 rpy=1.79407 -0.02832  2.14923, axis 0 0 1
- added joint right_2tip1: type revolute, parent right_2tip_base, child right_2tip1, axis 0 0 1, limit lower=-0.523599 upper=0.523599 effort=3.5 velocity=0.85
- added joint right_2tip2: type revolute, parent right_2tip1, child right_2tip2, origin xyz=0  0  0 rpy=1.57079  0       0, axis 0 0 1, limit lower=-0.349066 upper=1.50098 effort=3.5 velocity=0.85
- added joint right_2tip3: type revolute, parent right_2tip2, child right_2tip3, origin xyz=0.075  0     0 rpy=0  0  0, axis 0 0 1, limit lower=-0.174533 upper=1.76278 effort=1.75 velocity=0.85
- added joint right_2tip4: type revolute, parent right_2tip3, child right_2tip4, origin xyz=0.04  0    0 rpy=0       0      -1.57079, axis 0 0 1, limit lower=-0.174533 upper=1.76278 effort=1.75 velocity=0.85, mimic joint=right_2tip3 multiplier=1.0 offset=0
- added joint right_2tip_base: type fixed, parent right_arm7, child right_2tip_base, origin xyz=0.0482  0.2409  0.0236 rpy=-1.44842  0.11516  1.36812, axis 0 0 1
- added joint right_3middle1: type revolute, parent right_3middle_base, child right_3middle1, axis 0 0 1, limit lower=-0.523599 upper=0.523599 effort=3.5 velocity=0.85
- added joint right_3middle2: type revolute, parent right_3middle1, child right_3middle2, origin xyz=0  0  0 rpy=1.57079  0       0, axis 0 0 1, limit lower=-0.349066 upper=1.50098 effort=3.5 velocity=0.85
- added joint right_3middle3: type revolute, parent right_3middle2, child right_3middle3, origin xyz=0.075  0     0 rpy=0  0  0, axis 0 0 1, limit lower=-0.174533 upper=1.76278 effort=1.75 velocity=0.85
- added joint right_3middle4: type revolute, parent right_3middle3, child right_3middle4, origin xyz=0.04  0    0 rpy=0       0      -1.57079, axis 0 0 1, limit lower=-0.174533 upper=1.76278 effort=1.75 velocity=0.85, mimic joint=right_3middle3 multiplier=1.0 offset=0
- added joint right_3middle_base: type fixed, parent right_arm7, child right_3middle_base, origin xyz=0.0469   0.2353  -0.01629 rpy=-1.44842  0.11516  1.36812, axis 0 0 1
- added joint right_4ring1: type revolute, parent right_4ring_base, child right_4ring1, axis 0 0 1, limit lower=-0.523599 upper=0.523599 effort=3.5 velocity=0.85
- added joint right_4ring2: type revolute, parent right_4ring1, child right_4ring2, origin xyz=0  0  0 rpy=1.57079  0       0, axis 0 0 1, limit lower=-0.349066 upper=1.50098 effort=3.5 velocity=0.85
- added joint right_4ring3: type revolute, parent right_4ring2, child right_4ring3, origin xyz=0.075  0     0 rpy=0  0  0, axis 0 0 1, limit lower=-0.174533 upper=1.76278 effort=1.75 velocity=0.85
- added joint right_4ring4: type revolute, parent right_4ring3, child right_4ring4, origin xyz=0.04  0    0 rpy=0       0      -1.57079, axis 0 0 1, limit lower=-0.174533 upper=1.76278 effort=1.75 velocity=0.85, mimic joint=right_4ring3 multiplier=1.0 offset=0
- added joint right_4ring_base: type fixed, parent right_arm7, child right_4ring_base, origin xyz=0.0374  0.2299 -0.0623 rpy=-1.44842  0.11516  1.36812, axis 0 0 1
- added joint right_arm1: type revolute, parent torso4, child right_arm1, origin xyz=0.19   0.088 -0.256 rpy=3.14159  0.52359  3.14159, axis 0 0 1, limit lower=-2.96706 upper=2.96706 effort=150.0 velocity=0.85
- added joint right_arm2: type revolute, parent right_arm1, child right_arm2, origin xyz=0  0  0 rpy=1.57079  0       0, axis 0 0 1, limit lower=-2.0944 upper=2.0944 effort=150.0 velocity=0.85
- added joint right_arm3: type revolute, parent right_arm2, child right_arm3, origin xyz=0   0.4  0 rpy=0.35435 -1.57079 -1.92515, axis 0 0 1, limit lower=-2.96706 upper=2.96706 effort=150.0 velocity=0.85
- added joint right_arm4: type revolute, parent right_arm3, child right_arm4, origin xyz=0  0  0 rpy=1.57079  0       0, axis 0 0 1, limit lower=-2.0944 upper=2.0944 effort=150.0 velocity=0.85
- added joint right_arm5: type revolute, parent right_arm4, child right_arm5, origin xyz=0    0.39  0 rpy=1.57079  0      -3.14159, axis 0 0 1, limit lower=-2.96706 upper=2.96706 effort=150.0 velocity=0.85
- added joint right_arm6: type revolute, parent right_arm5, child right_arm6, origin xyz=0  0  0 rpy=0.39796 -1.57079  1.17283, axis 0 0 1, limit lower=-0.785398 upper=1.39626 effort=150.0 velocity=0.85
- added joint right_arm7: type revolute, parent right_arm6, child right_arm7, origin xyz=0  0  0 rpy=1.59992  1.57079  0.02912, axis 0 0 1, limit lower=-0.785398 upper=2.35619 effort=150.0 velocity=0.85
- added joint right_palm: type fixed, parent right_arm7, child right_palm, origin xyz=0  0.1011  0 rpy=1.57079 0.0 3.14159
- added joint torso1: type revolute, parent base_link, child torso1, origin xyz=0      0      0.6939 rpy=0  0  0, axis 0  0  1, limit lower=-1.74533 upper=3.31613 effort=150.0 velocity=0.85
- added joint torso2: type revolute, parent torso1, child torso2, origin xyz=0  0  0 rpy=-1.57079 -1.57079  0, axis 0  0  1, limit lower=-1.22173 upper=0.52360 effort=150.0 velocity=0.85
- added joint torso3: type revolute, parent torso2, child torso3, origin xyz=0.3  0   0 rpy=0  0  0, axis 0  0  1, limit lower=0.174533 upper=2.33874 effort=150.0 velocity=0.85
- added joint torso4: type revolute, parent torso3, child torso4, origin xyz=0.3  0   0 rpy=0  0  0, axis 0  0  1, limit lower=-1.57 upper=0.0 effort=150.0 velocity=0.85
