Commit message: Fix rollin_justin

File: multiverse/resources/robots/dlr/rollin_justin/urdf/rollin-justin.urdf (robot description, URDF)
Before this commit: robot rollin-justin, 63 links, 62 joints
Joints:
- removed joint head1
- removed joint head2
- removed joint left_1thumb1
- removed joint left_1thumb2
- removed joint left_1thumb3
- removed joint left_1thumb4
- removed joint left_1thumb_base
- removed joint left_2tip1
- removed joint left_2tip2
- removed joint left_2tip3
- removed joint left_2tip4
- removed joint left_2tip_base
- removed joint left_3middle1
- removed joint left_3middle2
- removed joint left_3middle3
- removed joint left_3middle4
- removed joint left_3middle_base
- removed joint left_4ring1
- removed joint left_4ring2
- removed joint left_4ring3
- removed joint left_4ring4
- removed joint left_4ring_base
- removed joint left_arm1
- removed joint left_arm2
- removed joint left_arm3
- removed joint left_arm4
- removed joint left_arm5
- removed joint left_arm6
- removed joint left_arm7
- removed joint left_palm
- removed joint right_1thumb1
- removed joint right_1thumb2
- removed joint right_1thumb3
- removed joint right_1thumb4
- removed joint right_1thumb_base
- removed joint right_2tip1
- removed joint right_2tip2
- removed joint right_2tip3
- removed joint right_2tip4
- removed joint right_2tip_base
- removed joint right_3middle1
- removed joint right_3middle2
- removed joint right_3middle3
- removed joint right_3middle4
- removed joint right_3middle_base
- removed joint right_4ring1
- removed joint right_4ring2
- removed joint right_4ring3
- removed joint right_4ring4
- removed joint right_4ring_base
- removed joint right_arm1
- removed joint right_arm2
- removed joint right_arm3
- removed joint right_arm4
- removed joint right_arm5
- removed joint right_arm6
- removed joint right_arm7
- removed joint right_palm
- removed joint torso1
- removed joint torso2
- removed joint torso3
- removed joint torso4
- added joint head1_joint: type revolute, parent torso4, child head1, origin xyz=0.235  0.088  0 rpy=1.57079  0       1.57079, axis 0  0  1, limit lower=-0.785398 upper=0.785398 effort=150.0 velocity=0.85
- added joint head2_joint: type revolute, parent head1, child head2, origin xyz=0  0  0 rpy=-1.57079  0       0, axis 0  0  1, limit lower=-0.436332 upper=0.785398 effort=150.0 velocity=0.85
- added joint left_1thumb1_joint: type revolute, parent left_1thumb_base, child left_1thumb1, axis 0 0 1, limit lower=-0.523599 upper=0.523599 effort=3.5 velocity=0.85
- added joint left_1thumb2_joint: type revolute, parent left_1thumb1, child left_1thumb2, origin xyz=0  0  0 rpy=1.57079  0       0, axis 0 0 1, limit lower=-0.349066 upper=1.50098 effort=3.5 velocity=0.85
- added joint left_1thumb3_joint: type revolute, parent left_1thumb2, child left_1thumb3, origin xyz=0.075  0     0 rpy=0  0  0, axis 0 0 1, limit lower=-0.174533 upper=1.76278 effort=1.75 velocity=0.85
- added joint left_1thumb4_joint: type revolute, parent left_1thumb3, child left_1thumb4, origin xyz=0.03999  0       0 rpy=0       0      -1.57079, axis 0 0 1, limit lower=-0.174533 upper=1.76278 effort=1.75 velocity=0.85, mimic joint=left_1thumb3_joint multiplier=1 offset=0
- added joint left_1thumb_base_joint: type fixed, parent left_arm7, child left_1thumb_base, origin xyz=-0.0504  0.2029 -0.0462 rpy=1.34429  0.02834  2.14927, axis 0 0 1
- added joint left_2tip1_joint: type revolute, parent left_2tip_base, child left_2tip1, axis 0 0 1, limit lower=-0.523599 upper=0.523599 effort=3.5 velocity=0.85
- added joint left_2tip2_joint: type revolute, parent left_2tip1, child left_2tip2, origin xyz=0  0  0 rpy=1.57079  0       0, axis 0 0 1, limit lower=-0.349066 upper=1.50098 effort=3.5 velocity=0.85
- added joint left_2tip3_joint: type revolute, parent left_2tip2, child left_2tip3, origin xyz=0.075  0     0 rpy=0  0  0, axis 0 0 1, limit lower=-0.174533 upper=1.76278 effort=1.75 velocity=0.85
- added joint left_2tip4_joint: type revolute, parent left_2tip3, child left_2tip4, origin xyz=0.04  0    0 rpy=0       0      -1.57079, axis 0 0 1, limit lower=-0.174533 upper=1.76278 effort=1.75 velocity=0.85, mimic joint=left_2tip3_joint multiplier=1.0 offset=0
- added joint left_2tip_base_joint: type fixed, parent left_arm7, child left_2tip_base, origin xyz=0.0482  0.2409 -0.0236 rpy=-1.69632 -0.11527  1.36803, axis 0 0 1
- added joint left_3middle1_joint: type revolute, parent left_3middle_base, child left_3middle1, axis 0 0 1, limit lower=-0.523599 upper=0.523599 effort=3.5 velocity=0.85
- added joint left_3middle2_joint: type revolute, parent left_3middle1, child left_3middle2, origin xyz=0  0  0 rpy=1.57079  0       0, axis 0 0 1, limit lower=-0.349066 upper=1.50098 effort=3.5 velocity=0.85
- added joint left_3middle3_joint: type revolute, parent left_3middle2, child left_3middle3, origin xyz=0.07499  0       0 rpy=0  0  0, axis 0 0 1, limit lower=-0.174533 upper=1.76278 effort=1.75 velocity=0.85
- added joint left_3middle4_joint: type revolute, parent left_3middle3, child left_3middle4, origin xyz=0.04  0    0 rpy=0       0      -1.57079, axis 0 0 1, limit lower=-0.174533 upper=1.76278 effort=1.75 velocity=0.85, mimic joint=left_3middle3_joint multiplier=1 offset=0
- added joint left_3middle_base_joint: type fixed, parent left_arm7, child left_3middle_base, origin xyz=0.0469   0.2353   0.01629 rpy=-1.69632 -0.11527  1.36803, axis 0 0 1
- added joint left_4ring1_joint: type revolute, parent left_4ring_base, child left_4ring1, axis 0 0 1, limit lower=-0.523599 upper=0.523599 effort=3.5 velocity=0.85
- added joint left_4ring2_joint: type revolute, parent left_4ring1, child left_4ring2, origin xyz=0  0  0 rpy=1.57079  0       0, axis 0 0 1, limit lower=-0.349066 upper=1.50098 effort=3.5 velocity=0.85
- added joint left_4ring3_joint: type revolute, parent left_4ring2, child left_4ring3, origin xyz=0.075  0     0 rpy=0  0  0, axis 0 0 1, limit lower=-0.174533 upper=1.76278 effort=1.75 velocity=0.85
- added joint left_4ring4_joint: type revolute, parent left_4ring3, child left_4ring4, origin xyz=0.04  0    0 rpy=0       0      -1.57079, axis 0 0 1, limit lower=-0.174533 upper=1.76278 effort=1.75 velocity=0.85, mimic joint=left_4ring3_joint multiplier=1 offset=0
- added joint left_4ring_base_joint: type fixed, parent left_arm7, child left_4ring_base, origin xyz=0.0374  0.2299  0.0623 rpy=-1.69632 -0.11527  1.36803, axis 0 0 1
- added joint left_arm1_joint: type revolute, parent torso4, child left_arm1, origin xyz=0.19   0.088  0.256 rpy=-3.14159  0.52359  0, axis 0  0  1, limit lower=-2.96706 upper=2.96706 effort=150.0 velocity=0.85
- added joint left_arm2_joint: type revolute, parent left_arm1, child left_arm2, origin xyz=0  0  0 rpy=1.57079  0       0, axis 0  0  1, limit lower=-2.0944 upper=2.0944 effort=150.0 velocity=0.85
- added joint left_arm3_joint: type revolute, parent left_arm2, child left_arm3, origin xyz=0  -0.4  0 rpy=-2.87979 -1.57079  1.30899, axis 0  0 1, limit lower=-2.96706 upper=2.96706 effort=150.0 velocity=0.85
- added joint left_arm4_joint: type revolute, parent left_arm3, child left_arm4, origin xyz=0  0  0 rpy=1.57079  0       0, axis 0 0 1, limit lower=-2.0944 upper=2.0944 effort=150.0 velocity=0.85
- added joint left_arm5_joint: type revolute, parent left_arm4, child left_arm5, origin xyz=0   -0.39  0 rpy=-1.57079  0       0, axis 0 0 1, limit lower=-2.96706 upper=2.96706 effort=150.0 velocity=0.85
- added joint left_arm6_joint: type revolute, parent left_arm5, child left_arm6, origin xyz=0  0  0 rpy=-0.71372  1.57079  0.85707, axis 0 0 1, limit lower=-0.785398 upper=1.39626 effort=150.0 velocity=0.85
- added joint left_arm7_joint: type revolute, parent left_arm6, child left_arm7, origin xyz=0  0  0 rpy=-1.11887 -1.57079 -0.45192, axis 0 0 1, limit lower=-0.785398 upper=2.35619 effort=150.0 velocity=0.85
- added joint left_palm_joint: type fixed, parent left_arm7, child left_palm, origin xyz=0  0.1011  0 rpy=1.57079 0.0 3.14159
- added joint right_1thumb1_joint: type revolute, parent right_1thumb_base, child right_1thumb1, axis 0 0 1, limit lower=-0.523599 upper=0.523599 effort=3.5 velocity=0.85
- added joint right_1thumb2_joint: type revolute, parent right_1thumb1, child right_1thumb2, origin xyz=0  0  0 rpy=1.57079  0       0, axis 0 0 1, limit lower=-0.349066 upper=1.50098 effort=3.5 velocity=0.85
- added joint right_1thumb3_joint: type revolute, parent right_1thumb2, child right_1thumb3, origin xyz=0.075  0     0 rpy=0  0  0, axis 0 0 1, limit lower=-0.174533 upper=1.76278 effort=1.75 velocity=0.85
- added joint right_1thumb4_joint: type revolute, parent right_1thumb3, child right_1thumb4, origin xyz=0.04  0    0 rpy=0       0      -1.57079, axis 0 0 1, limit lower=-0.174533 upper=1.76278 effort=1.75 velocity=0.85, mimic joint=right_1thumb3_joint multiplier=1.0 offset=0
- added joint right_1thumb_base_joint: type fixed, parent right_arm7, child right_1thumb_base, origin xyz=-0.0504  0.2029  0.0462 rpy=1.79407 -0.02832  2.14923, axis 0 0 1
- added joint right_2tip1_joint: type revolute, parent right_2tip_base, child right_2tip1, axis 0 0 1, limit lower=-0.523599 upper=0.523599 effort=3.5 velocity=0.85
- added joint right_2tip2_joint: type revolute, parent right_2tip1, child right_2tip2, origin xyz=0  0  0 rpy=1.57079  0       0, axis 0 0 1, limit lower=-0.349066 upper=1.50098 effort=3.5 velocity=0.85
- added joint right_2tip3_joint: type revolute, parent right_2tip2, child right_2tip3, origin xyz=0.075  0     0 rpy=0  0  0, axis 0 0 1, limit lower=-0.174533 upper=1.76278 effort=1.75 velocity=0.85
- added joint right_2tip4_joint: type revolute, parent right_2tip3, child right_2tip4, origin xyz=0.04  0    0 rpy=0       0      -1.57079, axis 0 0 1, limit lower=-0.174533 upper=1.76278 effort=1.75 velocity=0.85, mimic joint=right_2tip3_joint multiplier=1.0 offset=0
- added joint right_2tip_base_joint: type fixed, parent right_arm7, child right_2tip_base, origin xyz=0.0482  0.2409  0.0236 rpy=-1.44842  0.11516  1.36812, axis 0 0 1
- added joint right_3middle1_joint: type revolute, parent right_3middle_base, child right_3middle1, axis 0 0 1, limit lower=-0.523599 upper=0.523599 effort=3.5 velocity=0.85
- added joint right_3middle2_joint: type revolute, parent right_3middle1, child right_3middle2, origin xyz=0  0  0 rpy=1.57079  0       0, axis 0 0 1, limit lower=-0.349066 upper=1.50098 effort=3.5 velocity=0.85
- added joint right_3middle3_joint: type revolute, parent right_3middle2, child right_3middle3, origin xyz=0.075  0     0 rpy=0  0  0, axis 0 0 1, limit lower=-0.174533 upper=1.76278 effort=1.75 velocity=0.85
- added joint right_3middle4_joint: type revolute, parent right_3middle3, child right_3middle4, origin xyz=0.04  0    0 rpy=0       0      -1.57079, axis 0 0 1, limit lower=-0.174533 upper=1.76278 effort=1.75 velocity=0.85, mimic joint=right_3middle3_joint multiplier=1.0 offset=0
- added joint right_3middle_base_joint: type fixed, parent right_arm7, child right_3middle_base, origin xyz=0.0469   0.2353  -0.01629 rpy=-1.44842  0.11516  1.36812, axis 0 0 1
- added joint right_4ring1_joint: type revolute, parent right_4ring_base, child right_4ring1, axis 0 0 1, limit lower=-0.523599 upper=0.523599 effort=3.5 velocity=0.85
- added joint right_4ring2_joint: type revolute, parent right_4ring1, child right_4ring2, origin xyz=0  0  0 rpy=1.57079  0       0, axis 0 0 1, limit lower=-0.349066 upper=1.50098 effort=3.5 velocity=0.85
- added joint right_4ring3_joint: type revolute, parent right_4ring2, child right_4ring3, origin xyz=0.075  0     0 rpy=0  0  0, axis 0 0 1, limit lower=-0.174533 upper=1.76278 effort=1.75 velocity=0.85
- added joint right_4ring4_joint: type revolute, parent right_4ring3, child right_4ring4, origin xyz=0.04  0    0 rpy=0       0      -1.57079, axis 0 0 1, limit lower=-0.174533 upper=1.76278 effort=1.75 velocity=0.85, mimic joint=right_4ring3_joint multiplier=1.0 offset=0
- added joint right_4ring_base_joint: type fixed, parent right_arm7, child right_4ring_base, origin xyz=0.0374  0.2299 -0.0623 rpy=-1.44842  0.11516  1.36812, axis 0 0 1
- added joint right_arm1_joint: type revolute, parent torso4, child right_arm1, origin xyz=0.19   0.088 -0.256 rpy=3.14159  0.52359  3.14159, axis 0 0 1, limit lower=-2.96706 upper=2.96706 effort=150.0 velocity=0.85
- added joint right_arm2_joint: type revolute, parent right_arm1, child right_arm2, origin xyz=0  0  0 rpy=1.57079  0       0, axis 0 0 1, limit lower=-2.0944 upper=2.0944 effort=150.0 velocity=0.85
- added joint right_arm3_joint: type revolute, parent right_arm2, child right_arm3, origin xyz=0   0.4  0 rpy=0.35435 -1.57079 -1.92515, axis 0 0 1, limit lower=-2.96706 upper=2.96706 effort=150.0 velocity=0.85
- added joint right_arm4_joint: type revolute, parent right_arm3, child right_arm4, origin xyz=0  0  0 rpy=1.57079  0       0, axis 0 0 1, limit lower=-2.0944 upper=2.0944 effort=150.0 velocity=0.85
- added joint right_arm5_joint: type revolute, parent right_arm4, child right_arm5, origin xyz=0    0.39  0 rpy=1.57079  0      -3.14159, axis 0 0 1, limit lower=-2.96706 upper=2.96706 effort=150.0 velocity=0.85
- added joint right_arm6_joint: type revolute, parent right_arm5, child right_arm6, origin xyz=0  0  0 rpy=0.39796 -1.57079  1.17283, axis 0 0 1, limit lower=-0.785398 upper=1.39626 effort=150.0 velocity=0.85
- added joint right_arm7_joint: type revolute, parent right_arm6, child right_arm7, origin xyz=0  0  0 rpy=1.59992  1.57079  0.02912, axis 0 0 1, limit lower=-0.785398 upper=2.35619 effort=150.0 velocity=0.85
- added joint right_palm_joint: type fixed, parent right_arm7, child right_palm, origin xyz=0  0.1011  0 rpy=1.57079 0.0 3.14159
- added joint torso1_joint: type revolute, parent base_link, child torso1, origin xyz=0      0      0.6939 rpy=0  0  0, axis 0  0  1, limit lower=-1.74533 upper=3.31613 effort=150.0 velocity=0.85
- added joint torso2_joint: type revolute, parent torso1, child torso2, origin xyz=0  0  0 rpy=-1.57079 -1.57079  0, axis 0  0  1, limit lower=-1.22173 upper=0.52360 effort=150.0 velocity=0.85
- added joint torso3_joint: type revolute, parent torso2, child torso3, origin xyz=0.3  0   0 rpy=0  0  0, axis 0  0  1, limit lower=0.174533 upper=2.33874 effort=150.0 velocity=0.85
- added joint torso4_joint: type revolute, parent torso3, child torso4, origin xyz=0.3  0   0 rpy=0  0  0, axis 0  0  1, limit lower=-1.57 upper=0.0 effort=150.0 velocity=0.85
