Commit message: Change virual joints to fixed

File: multiverse/resources/robots/pr2/pr2.urdf (robot description, URDF)
Before this commit: robot pr2, 89 links, 88 joints
Joints:
- joint l_gripper_joint: axis 0.0 1.0 0.0 -> (none); limit lower=0.0 upper=0.09000000357627869 effort=1000.0 velocity=0.20000000298023224 -> (none); type prismatic -> fixed
- joint l_gripper_motor_screw_joint: axis 0.0 1.0 0.0 -> (none); type continuous -> fixed
- joint l_gripper_motor_slider_joint: axis 1.0 0.0 0.0 -> (none); limit lower=-0.10000000149011612 upper=0.10000000149011612 effort=1000.0 velocity=0.20000000298023224 -> (none); type prismatic -> fixed
- joint r_gripper_joint: axis 0.0 1.0 0.0 -> (none); limit lower=0.0 upper=0.09000000357627869 effort=1000.0 velocity=0.20000000298023224 -> (none); type prismatic -> fixed
- joint r_gripper_motor_screw_joint: axis 0.0 1.0 0.0 -> (none); type continuous -> fixed
- joint r_gripper_motor_slider_joint: axis 1.0 0.0 0.0 -> (none); limit lower=-0.10000000149011612 upper=0.10000000149011612 effort=1000.0 velocity=0.20000000298023224 -> (none); type prismatic -> fixed
- joint torso_lift_motor_screw_joint: axis 0.0 0.0 1.0 -> (none); type continuous -> fixed
