Commit message: Update

File: Demos/1_TiagoDualInApartment/assets/urdf/iai_tiago_with_ros2_control_velocity.urdf (robot description, URDF)
Before this commit: robot base_footprint, 68 links, 67 joints
Links:
- added link gripper_left_tool_frame
- added link gripper_right_tool_frame
Joints:
- added joint gripper_left_tool_frame_joint: type fixed, parent gripper_left_base_link, child gripper_left_tool_frame, origin xyz=0 0 0.2
- added joint gripper_right_tool_frame_joint: type fixed, parent gripper_right_base_link, child gripper_right_tool_frame, origin xyz=0 0 0.2
